File: stereo_mix/stereo_mix.sch (EAGLE design)
At the start: 16 parts, among them U1 THONKICONNNEW, U2 THONKICONNNEW, U3 THONKICONNNEW, U4 THONKICONNNEW, U5 THONKICONNNEW, U6 THONKICONNNEW, U7 THONKICONNNEW, U8 THONKICONNNEW

Commit message: Start implementation of stereo_mixer
Parts:
- added U10, U11, U12, U13, U14, U15, U16, U17, U18, U19, U20, U9: THONKICONNNEW, MusicThingModular:THONKICONNNEW
- added UB_L, UB_R: (no value), jumper:JP2E
- VR2, VR3, VR4: SPICEPREFIX (none) -> J
- VR5, VR6, VR7, VR8: device MusicThingModular:ALPHA-9MM-DUALPOT -> MusicThingModular:9MM_SNAP-IN_POT_; SPICEPREFIX (none) -> J
Connections:
- new net N$17: U4.TIP, VR2.E
- new net N$18: U11.TIP, VR5.E
- new net N$19: VR5.A
- new net N$20: VR6.S
- new net N$21: U12.TIP, VR6.E
- new net N$22: U13.TIP, U14.SWITCH
- new net N$23: U14.TIP
- new net N$24: VR7.S
- new net N$25: U15.TIP, VR7.E
- new net N$26: VR7.A
- new net N$27: VR8.S
- new net N$28: U16.TIP, VR8.E
- new net N$29: U17.TIP
- new net N$30: U18.TIP
- new net N$31: U18.SWITCH, U20.TIP
- new net N$32: U17.SWITCH, U19.TIP
- new net REF_10: U12.SWITCH, U16.SWITCH, U4.SWITCH, U8.SWITCH
- new net REF_5: U11.SWITCH, U15.SWITCH, U3.SWITCH, U7.SWITCH
- net GND: now also U1.SLEEVE, U10.SLEEVE, U11.SLEEVE, U12.SLEEVE, U13.SLEEVE, U14.SLEEVE, U15.SLEEVE, U16.SLEEVE, U17.SLEEVE, U18.SLEEVE, U19.SLEEVE, U2.SLEEVE, U20.SLEEVE, U3.SLEEVE, U4.SLEEVE, U5.SLEEVE, U6.SLEEVE, U7.SLEEVE, U8.SLEEVE, U9.SLEEVE, VR2.A, VR4.A, VR6.A, VR8.A; no longer VR1.S, VR2.S, VR3.S, VR4.S, VR5G$1.A, VR5G$2.A, VR6G$1.A, VR6G$2.A, VR7G$1.A, VR7G$2.A, VR8G$1.A, VR8G$2.A
- net N$1: no longer VR1.A, VR5G$1.E
- net N$10: now also U7.TIP, VR3.E; no longer VR5G$1.S
- net N$11: now also VR3.A; no longer VR5G$2.S
- net N$12: now also VR4.S; no longer VR6G$1.S
- net N$13: now also U8.TIP, VR4.E; no longer VR7G$1.S
- net N$14: now also U10.SWITCH, U9.TIP; no longer VR7G$2.S
- net N$15: now also U10.TIP; no longer VR8G$1.S
- net N$16: now also VR5.S; no longer VR8G$2.S
- net N$2: now also U2.TIP; no longer U3.TIP, U4.SWITCH, VR2.A, VR6G$1.E
- net N$3: now also VR1.S; no longer U5.TIP, U6.SWITCH, VR3.A, VR7G$1.E
- net N$4: now also U5.TIP, U6.SWITCH; no longer U7.TIP, U8.SWITCH, VR4.A, VR8G$1.E
- net N$5: now also U3.TIP, VR1.E; no longer VR6G$2.S
- net N$6: now also VR1.A; no longer U2.TIP, VR1.E, VR5G$2.E
- net N$7: now also VR2.S; no longer U4.TIP, VR2.E, VR6G$2.E
- net N$8: no longer VR3.E, VR7G$2.E
- net N$9: now also VR3.S; no longer U8.TIP, VR4.E, VR8G$2.E
