File: stereo_mix/stereo_mix_back.sch (EAGLE design)
At the start: 30 parts, among them U1 THONKICONNNEW, U10 THONKICONNNEW, U11 THONKICONNNEW, U12 THONKICONNNEW, U13 THONKICONNNEW, U14 THONKICONNNEW, U15 THONKICONNNEW, U16 THONKICONNNEW, U17 THONKICONNNEW, U18 THONKICONNNEW, U19 THONKICONNNEW, U2 THONKICONNNEW, U20 THONKICONNNEW, U3 THONKICONNNEW, U4 THONKICONNNEW, U5 THONKICONNNEW, U6 THONKICONNNEW, U7 THONKICONNNEW, U8 THONKICONNNEW, U9 THONKICONNNEW

Commit message: Make stereo mix a two layer board
Parts:
- removed U1, U10, U11, U12, U13, U14, U15, U16, U17, U18, U19, U2, U20, U3, U4, U5, U6, U7, U8, U9: THONKICONNNEW, MusicThingModular:THONKICONNNEW
- removed UB_L, UB_R: (no value), jumper:JP2E
- removed VR1, VR2, VR3, VR4, VR5, VR6, VR7, VR8: (no value), MusicThingModular:9MM_SNAP-IN_POT_
- added AUX_IN, AUX_OUT, BAL_L, BAL_R: (no value), jumper:JP2E
- added C5: EURO_POWER_LOCKFAT-LOCK, MusicThingModular:EURO_POWER_LOCKFAT-LOCK
- added D1, D2: 1N4001, adafruit:DIODESMA
- added IC1: TL084PW, op-amp:TL084PW
- added IC6: TL082PW, op-amp:TL082PW
- added JP1: (no value), pinhead:PINHD-1X20
- added JP2: (no value), pinhead:PINHD-1X5
- added JP4: (no value), pinhead:PINHD-1X9
- added R10, R13, R14, R17, R18, R19, R20, R3, R4, R5, R6, R7, R8, R9: 100k, rcl:R-EU_R0603
- added R12, R16: 24k, rcl:R-EU_R0603
- added R21: (no value), rcl:R-EU_R0603
- added R22: 680R, rcl:R-EU_R0603
- added RN1: CTS742C083, resistor-net:CTS742C083
- added U21: TEXAS_INSTRUMENTS_LM4040C5IDBZR, lm4040:TEXAS_INSTRUMENTS_LM4040C5IDBZR
- added U22: TEXAS_INSTRUMENTS_LM4040C10IDBZR, lm4040:TEXAS_INSTRUMENTS_LM4040C10IDBZR
Connections:
- removed net N$19: VR5.A
- removed net N$2: U2.TIP
- removed net N$25: U15.TIP, VR7.E
- removed net N$31: U18.SWITCH, U20.TIP
- new net +12V: D1.C, IC1P.V+, IC1SUPPLY.V+, IC6P.V+, JP1.1, R13.E, R21.2, R22.2, R5.1
- new net -12V: D2.A, IC1P.V-, IC1SUPPLY.V-, IC6P.V-, JP1.19, R13.A, R18.2
- new net 1_IN_L: JP1.2
- new net 1_IN_R: JP1.3
- new net 1_PAN_ATT_R: JP1.6
- new net 1_PAN_ATT_W: JP1.5
- new net 1_PAN_CV_IN: JP1.4
- new net 1_VOLUME_CV: JP1.7
- new net 2_IN_L: JP1.8
- new net 2_IN_R: JP1.9
- new net 2_PAN_ATT_R: JP1.12
- new net 2_PAN_ATT_W: JP1.11
- new net 2_PAN_CV_IN: JP1.10
- new net 2_VOLUME_CV: JP1.13
- new net 3_IN_L: JP1.14
- new net 3_IN_R: JP1.15
- new net 3_PAN_ATT_R: JP1.18
- new net 3_PAN_ATT_W: JP1.17
- new net 3_PAN_CV_IN: JP1.16
- new net 3_VOLUME_CV: JP4.1
- new net 4_IN_L: JP4.2
- new net 4_IN_R: JP4.3
- new net 4_PAN_ATT_R: JP4.6
- new net 4_PAN_ATT_W: JP4.5
- new net 4_PAN_CV_IN: JP4.4
- new net 4_VOLUME_CV: JP4.7
- new net AUX_IN_L: AUX_IN.1, R19.1
- new net AUX_IN_R: AUX_IN.2, R20.1
- new net BAL_N_L: BAL_L.2, IC6B.OUT, R14.2
- new net BAL_N_R: BAL_R.2, IC6A.OUT, R18.2
- new net BAL_P_L: BAL_L.1, IC1C.OUT, R12.2, R13.1
- new net BAL_P_R: BAL_R.1, IC1A.OUT, R16.2, R17.1
- new net BYPASS_L: AUX_OUT.1, IC1B.OUT, JP2.3, RN1.8
- new net BYPASS_R: AUX_OUT.2, IC1D.OUT, JP2.4, RN1.5
- new net IN_L: R4.1
- new net IN_R: R22.1
- new net N$33: R5.1
- new net N$35: R6.1
- new net N$37: R7.1
- new net N$38: R8.1
- new net N$39: R9.1
- new net N$40: R10.1
- new net N$41: C5.1
- new net N$42: C5.2, IC1A.+IN, R16.1, RN1.3
- new net N$43: IC6A.+IN, IC6B.+IN, R17.2, R18.1, RN1.3, RN1.4
- new net N$45: IC6B.-IN, R13.2, R14.1, RN1.1, RN1.2
- new net N$47: C5.+12V, D1.A, IC6A.-IN
- new net N$48: C5.-12V, D2.C
- new net N$50: IC6A.+IN
- new net OUT_L: JP2.1, RN1.7
- new net OUT_R: JP2.2, RN1.6
- new net PAN_CV: RN1.7
- new net PAN_CV_L: IC6B.OUT, R7.1, RN1.8
- new net PAN_CV_R: IC6A.OUT
- new net SUM_L: IC1B.+IN, R19.2, R3.2, R5.2, R7.2, R9.2, RN1.1
- new net SUM_R: IC1D.-IN, R10.2, R20.2, R4.2, R6.2, R8.2, RN1.4
- net GND: now also AUX_IN.3, AUX_OUT.3, BAL_L.3, BAL_R.3, C5.GND, IC1A.-IN, IC1B.-IN, IC1C.-IN, IC1D.+IN, IC6A.-IN, IC6B.+IN, JP1.20, JP2.5, R16.1, R20.1, R21.1, R3.1, RN1.5, U21.ANODE, U22.ANODE; no longer U1.SLEEVE, U10.SLEEVE, U11.SLEEVE, U12.SLEEVE, U13.SLEEVE, U14.SLEEVE, U15.SLEEVE, U16.SLEEVE, U17.SLEEVE, U18.SLEEVE, U19.SLEEVE, U2.SLEEVE, U20.SLEEVE, U3.SLEEVE, U4.SLEEVE, U5.SLEEVE, U6.SLEEVE, U7.SLEEVE, U8.SLEEVE, U9.SLEEVE, VR2.A, VR4.A, VR6.A, VR8.A
- net N$1: now also IC1OTA1.IN_N; no longer U1.TIP, U2.SWITCH
- net N$10: now also R8.1, R9.2; no longer U7.TIP, VR3.E
- net N$11: now also R10.1, R8.2; no longer VR3.A
- net N$12: now also R12.2, R14.1; no longer VR4.S
- net N$13: now also R10.2; no longer U8.TIP, VR4.E
- net N$14: now also R12.1, R13.S; no longer U10.SWITCH, U9.TIP
- net N$15: now also R16.2; no longer U10.TIP
- net N$16: now also R14.2; no longer VR5.S
- net N$17: now also R17.2; no longer U4.TIP, VR2.E
- net N$18: now also R17.1, R18.1; no longer U11.TIP, VR5.E
- net N$20: now also IC1OTA2.IN_N, R19.2; no longer VR6.S
- net N$21: now also R19.1, R20.2; no longer U12.TIP, VR6.E
- net N$22: now also IC1OTA2.IN_P, R21.2, R22.2; no longer U13.TIP, U14.SWITCH
- net N$23: now also IC1OTA2.I_DIODE; no longer U14.TIP
- net N$24: now also IC1OTA2.I_BIAS; no longer VR7.S
- net N$26: now also D2.A; no longer VR7.A
- net N$27: now also D2.C; no longer VR8.S
- net N$28: now also IC1OTA2.OUT; no longer U16.TIP, VR8.E
- net N$29: now also R3.1; no longer U17.TIP
- net N$3: now also IC1OTA1.IN_P, R3.2, R4.2; no longer VR1.S
- net N$30: now also R4.1; no longer U18.TIP
- net N$32: now also IC1C.+IN, R12.1, RN1.2; no longer U17.SWITCH, U19.TIP
- net N$4: now also IC1OTA1.I_BIAS, R6.2; no longer U5.TIP, U6.SWITCH
- net N$5: now also IC1OTA1.I_DIODE, R5.2; no longer U3.TIP, VR1.E
- net N$6: now also R6.1; no longer VR1.A
- net N$7: now also D1.A; no longer VR2.S
- net N$8: now also D1.C, R7.2; no longer U6.TIP
- net N$9: now also IC1OTA1.OUT, R9.1; no longer VR3.S
- net REF_10: now also JP4.9, R22.1, U22.CATHODE; no longer U12.SWITCH, U16.SWITCH, U4.SWITCH, U8.SWITCH
- net REF_5: now also JP4.8, R21.1, RN1.6, U21.CATHODE; no longer U11.SWITCH, U15.SWITCH, U3.SWITCH, U7.SWITCH
