File: vca2/hardware_design/vca2.sch (EAGLE design)
At the start: 112 parts, among them IC1 LM13700M, IC2 NCS20074D, IC3 TL074D, IC4 TL072D, IC5 NCS20074D, T1 2N3906, T2 BC847BS, T3 2N3906, T4 2N3906, T5 BC847BS, T6 2N3906

Commit message: New version of vca2 with manufacturing parts. This is the first dirty version!!!!!
Parts:
- removed C6, C7: 22uF, rcl:CPOL-EUC
- removed IC3: TL074D, linear:TL074D
- added C22, C23: 100nF, jhbruhn-cr:C-EUC0402
- added C24, C25: 10uF, rcl:CPOL-EUA/3216-18W
- added U1, U2: TL072CD, jhbruhn-opamp:TL072CD
- C1: device MusicThingModular:EURO_POWER_LOCKFAT-LOCK -> jhbruhn-physical:EURO_POWER_LOCKFAT-LOCK
- C10, C11, C12, C13, C14, C15, C16, C17, C18, C19, C2, C20, C21, C3, C4, C5, C8, C9: device rcl:C-EUC0603 -> jhbruhn-cr:C-EUC0402
- IC1: device ota:LM13700M -> jhbruhn-ota:LM13700M
- IC4: value TL072D -> TL072CD; device linear:TL072D -> jhbruhn-opamp:TL072CD
- R1, R10, R11, R12, R13, R15, R16, R17, R19, R2, R20, R21, R22, R23, R24, R25, R26, R27, R28, R29, R3, R30, R31, R32, R33, R34, R35, R36, R38, R39, R4, R40, R42, R43, R44, R45, R46, R47, R48, R49, R5, R50, R51, R52, R53, R54, R55, R6, R7, R8, R9: device rcl:R-EU_R0603 -> jhbruhn-cr:R-EU_R0402
- R14, R37: value 600R -> 680R; device rcl:R-EU_R0603 -> jhbruhn-cr:R-EU_R0402
- U$1, U$2, U$3, U$4, U$6, U$7, U$8, U$9: device thonkiconn:WQP-PJ301M-12_JACK -> jhbruhn-physical:WQP-PJ301M-12_JACK
- VR1, VR2, VR3, VR4: device MusicThingModular:9MM_SNAP-IN_POT_ -> jhbruhn-physical:9MM_SNAP-IN_POT_
Connections:
- net +12V: now also C22.1, C24.+, U1P.V+, U2P.V+; no longer C6.+, IC3P.V+
- net -12V: now also C23.2, C25.-, U1P.V-, U2P.V-; no longer C7.-, IC3P.V-
- net GND: now also C22.2, C23.1, C24.-, C25.+; no longer C6.-, C7.+
- net N$19: now also U1B.+IN; no longer IC3B.+IN
- net N$20: now also U1B.-IN; no longer IC3B.-IN
- net N$22: now also U1B.OUT; no longer IC3B.OUT
- net N$23: now also U1A.-IN, U1A.OUT; no longer IC3A.-IN, IC3A.OUT
- net N$24: now also U1A.+IN; no longer IC3A.+IN
- net N$45: now also U2B.-IN; no longer IC3D.-IN
- net N$46: now also U2B.+IN; no longer IC3D.+IN
- net N$47: now also U2B.OUT; no longer IC3D.OUT
- net N$49: now also U2A.-IN, U2A.OUT; no longer IC3C.-IN, IC3C.OUT
- net N$50: now also U2A.+IN; no longer IC3C.+IN
Other:
- moved on the sheet: U$1, U$2, U$3, U$4, U$6, U$7, U$8, U$9
