File: out/hardware_design/pcb/out.brd (EAGLE design)
At the start: 60 x 60 mm, 77 parts, among them T1 MMBT3904, T2 MMBT3904, T3 MMBT3904, U1 TL072CD, U2 TL072CD, U3 TL072CD, U4 NE5532D, U5 NE5532D

Commit message: Fix out oderso, implement menu scrolling i guess
Connections:
- net -12V: now also D2.A, D4.A; no longer D2.C, D4.C
- net N$1: now also D2.C; no longer D2.A
- net N$2: now also D4.C; no longer D4.A
Routing:
- net -12V: track 112.1 -> 105.5 mm
Changed lines of the file:
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@@
 <drawing>
 <settings>
-<setting alwaysvectorfont="yes"/>
+<setting alwaysvectorfont="no"/>
 <setting verticaltext="up"/>
 </settings>
@@
 <contactref element="R19" pad="1"/>
 <contactref element="D1" pad="A"/>
-<contactref element="D2" pad="A"/>
 <contactref element="C5" pad="2"/>
 <contactref element="R8" pad="2"/>
@@
 <wire x1="48.006" y1="38.0619" x2="48.006" y2="37.2618" width="0.254" layer="1"/>
 <wire x1="48.006" y1="37.2618" x2="48.006" y2="34.29" width="0.254" layer="1"/>
-<wire x1="48.006" y1="34.29" x2="47.99" y2="34.29" width="0.254" layer="1"/>
 <wire x1="48.006" y1="38.0619" x2="47.99" y2="38.1" width="0.254" layer="1"/>
 <wire x1="21.717" y1="38.6334" x2="24.1173" y2="38.6334" width="0.254" layer="1"/>
@@
 <wire x1="26.7462" y1="38.862" x2="27.0891" y2="39.2049" width="0.254" layer="1"/>
 <wire x1="26.7462" y1="38.862" x2="26.67" y2="38.75" width="0.254" layer="1"/>
+<contactref element="D2" pad="C"/>
+<wire x1="48.006" y1="34.29" x2="45.99" y2="34.29" width="0" layer="19" extent="1-1"/>
 </signal>
 <signal name="N$2">
@@
 <contactref element="R21" pad="1"/>
 <contactref element="D3" pad="A"/>
-<contactref element="D4" pad="A"/>
 <contactref element="R10" pad="2"/>
 <contactref element="C4" pad="2"/>
 <wire x1="48.006" y1="28.0035" x2="50.292" y2="28.0035" width="0.254" layer="1"/>
 <wire x1="50.292" y1="28.0035" x2="50.3" y2="27.94" width="0.254" layer="1"/>
-<wire x1="48.006" y1="28.0035" x2="47.99" y2="27.94" width="0.254" layer="1"/>
 <wire x1="48.006" y1="27.8892" x2="48.006" y2="27.2034" width="0.254" layer="1"/>
 <wire x1="48.006" y1="27.2034" x2="48.006" y2="24.2316" width="0.254" layer="1"/>
 <wire x1="48.006" y1="24.2316" x2="47.99" y2="24.13" width="0.254" layer="1"/>
-<wire x1="48.006" y1="27.8892" x2="47.99" y2="27.94" width="0.254" layer="1"/>
 <wire x1="26.5176" y1="28.4607" x2="24.2316" y2="28.4607" width="0.254" layer="1"/>
 <wire x1="26.6319" y1="28.575" x2="26.5176" y2="28.4607" width="0.254" layer="1"/>
@@
 <wire x1="26.7462" y1="28.6893" x2="27.0891" y2="29.0322" width="0.254" layer="1"/>
 <wire x1="26.7462" y1="28.6893" x2="26.67" y2="28.59" width="0.254" layer="1"/>
+<contactref element="D4" pad="C"/>
+<wire x1="48.006" y1="27.8892" x2="48.006" y2="28.0035" width="0" layer="19" extent="1-1"/>
+<wire x1="45.99" y1="27.94" x2="48.006" y2="28.0035" width="0" layer="19" extent="1-1"/>
 </signal>
 <signal name="N$3">
@@
 <contactref element="C19" pad="2"/>
 <contactref element="C20" pad="2"/>
-<contactref element="D4" pad="C"/>
-<contactref element="D2" pad="C"/>
 <contactref element="D6" pad="A"/>
 <contactref element="C10" pad="-"/>
-<wire x1="45.9486" y1="34.29" x2="45.9486" y2="28.0035" width="0.4064" layer="1"/>
-<wire x1="45.9486" y1="28.0035" x2="45.99" y2="27.94" width="0.4064" layer="1"/>
-<wire x1="45.9486" y1="34.29" x2="45.99" y2="34.29" width="0.4064" layer="1"/>
 <wire x1="38.862" y1="51.0921" x2="38.862" y2="49.6062" width="0.4064" layer="1"/>
 <wire x1="39.2049" y1="51.435" x2="38.862" y2="51.0921" width="0.4064" layer="1"/>
@@
 <wire x1="40.005" y1="41.0337" x2="40.005" y2="36.6903" width="0.4064" layer="16"/>
 <wire x1="37.8333" y1="43.2054" x2="40.005" y2="41.0337" width="0.4064" layer="16"/>
-<wire x1="45.8343" y1="34.4043" x2="45.99" y2="34.29" width="0.4064" layer="1"/>
 <wire x1="40.3479" y1="9.6012" x2="40.3479" y2="12.6873" width="0.4064" layer="1"/>
 <wire x1="39.6621" y1="8.9154" x2="40.3479" y2="9.6012" width="0.4064" layer="1"/>
@@
 <via x="16.002" y="25.146" extent="1-16" drill="0.3048"/>
 <via x="38.9763" y="13.9446" extent="1-16" drill="0.3048"/>
+<contactref element="D4" pad="A"/>
+<contactref element="D2" pad="A"/>
+<wire x1="45.8343" y1="34.4043" x2="47.99" y2="34.29" width="0" layer="19" extent="1-1"/>
+<wire x1="47.99" y1="27.94" x2="47.99" y2="34.29" width="0" layer="19" extent="1-1"/>
 </signal>
 <signal name="N$40">
