File: vca/hardware_design/vca.sch (EAGLE design)
At the start: 69 parts, among them IC1 LM13700M, IC2 TL074D

Commit message: Rename vca2 to vca, remove vca
Parts:
- removed C6, C7: 22uF, rcl:CPOL-EUC
- removed U$10, U$5: INSTRUO_TOGGLE_ON_OFF_ON, Pure LFO:INSTRUO_TOGGLE_ON_OFF_ON
- added C10, C11, C14, C15: 22pF, jhbruhn-cr:C-EUC0402
- added C12, C13, C8, C9: 100pF, jhbruhn-cr:C-EUC0402
- added C16, C17, C18, C19, C20, C21, C22, C23: 100nF, jhbruhn-cr:C-EUC0402
- added C24, C25: 10uF, rcl:CPOL-EUA/3216-18W
- added D3, D4: 1N4148-2, adafruit:DIODESOD-123
- added FD1, FD2, FD3, FD4: FIDUCIAL1X2, SparkFun-Aesthetics:FIDUCIAL1X2
- added IC4, U1, U2: TL072CD, jhbruhn-opamp:TL072CD
- added IC5: NCS20074D, ncs20074:NCS20074D
- added LOGO1: OSHW-LOGOM, SparkFun-Aesthetics:OSHW-LOGOM
- added R43: 68k, jhbruhn-cr:R-EU_R0402
- added R44, R47: 1k, jhbruhn-cr:R-EU_R0402
- added R45: 15k, jhbruhn-cr:R-EU_R0402
- added R46: 680k, jhbruhn-cr:R-EU_R0402
- added R48, R49, R50, R51, R52, R53: 100k, jhbruhn-cr:R-EU_R0402
- added R54: 10k, jhbruhn-cr:R-EU_R0402
- added R55: 50k, jhbruhn-cr:R-EU_R0402
- added SJ1, SJ2, SJ3, SJ4: (no value), jumper:SJ
- added T5: BC847BS, nxp_60:BC847BS
- added T6: 2N3906, transistor-neu-to92:MMBT3906LT1-PNP-SOT23-BEC
- added VR3, VR4: 100k, jhbruhn-physical:9MM_SNAP-IN_POT_
- C1: device MusicThingModular:EURO_POWER_LOCKFAT-LOCK -> jhbruhn-physical:EURO_POWER_LOCKFAT-LOCK
- C2, C3, C4, C5: device rcl:C-EUC0603 -> jhbruhn-cr:C-EUC0402
- IC1: device ota:LM13700M -> jhbruhn-ota:LM13700M
- IC2: value TL074D -> NCS20074D; device linear:TL074D -> ncs20074:NCS20074D
- R1, R21, R24: value 100k -> 1k; device rcl:R-EU_R0603 -> jhbruhn-cr:R-EU_R0402
- R10: value 470 -> 10k; device rcl:R-EU_R0603 -> jhbruhn-cr:R-EU_R0402
- R11: value 100k -> 10M; device rcl:R-EU_R0603 -> jhbruhn-cr:R-EU_R0402
- R12: value 100k -> 1k5; device rcl:R-EU_R0603 -> jhbruhn-cr:R-EU_R0402
- R13: value 2k -> 100k; device rcl:R-TRIMM64W -> jhbruhn-cr:R-EU_R0402
- R14: value 150 -> 680R; device rcl:R-EU_R0603 -> jhbruhn-cr:R-EU_R0402
- R15: value 2M -> 47k; device rcl:R-EU_R0603 -> jhbruhn-cr:R-EU_R0402
- R16: value 470k -> 680R; device rcl:R-EU_R0603 -> jhbruhn-cr:R-EU_R0402
- R17: value 47k -> 1M; device rcl:R-EU_R0603 -> jhbruhn-cr:R-EU_R0402
- R18: value 4k7 -> 100k; device rcl:R-EU_R0603 -> rcl:R-TRIMM64W
- R19: value 1k -> 100k; device rcl:R-EU_R0603 -> jhbruhn-cr:R-EU_R0402
- R2, R3: value 100k -> 1M; device rcl:R-EU_R0603 -> jhbruhn-cr:R-EU_R0402
- R20: value 20k -> 68k; device rcl:R-EU_R0603 -> jhbruhn-cr:R-EU_R0402
- R22: value 100k -> 15k; device rcl:R-EU_R0603 -> jhbruhn-cr:R-EU_R0402
- R23: value 100k -> 680k; device rcl:R-EU_R0603 -> jhbruhn-cr:R-EU_R0402
- R25, R26: value 2k -> 1M; device rcl:R-EU_R0603 -> jhbruhn-cr:R-EU_R0402
- R27: value 120k -> 100k; device rcl:R-EU_R0603 -> jhbruhn-cr:R-EU_R0402
- R28, R5: value 2k -> 100k; device rcl:R-EU_R0603 -> jhbruhn-cr:R-EU_R0402
- R29: value 100k -> 220R; device rcl:R-EU_R0603 -> jhbruhn-cr:R-EU_R0402
- R30: value 470 -> 220R; device rcl:R-EU_R0603 -> jhbruhn-cr:R-EU_R0402
- R31: value 100k -> 56k; device rcl:R-EU_R0603 -> jhbruhn-cr:R-EU_R0402
- R32, R9: value 100k -> 33k; device rcl:R-EU_R0603 -> jhbruhn-cr:R-EU_R0402
- R33: value 2k -> 10k; device rcl:R-TRIMM64W -> jhbruhn-cr:R-EU_R0402
- R34: value 150 -> 10M; device rcl:R-EU_R0603 -> jhbruhn-cr:R-EU_R0402
- R35: value 2M -> 1k5; device rcl:R-EU_R0603 -> jhbruhn-cr:R-EU_R0402
- R36: value 470k -> 100k; device rcl:R-EU_R0603 -> jhbruhn-cr:R-EU_R0402
- R37: value 47k -> 680R; device rcl:R-EU_R0603 -> jhbruhn-cr:R-EU_R0402
- R38: value 4k7 -> 47k; device rcl:R-EU_R0603 -> jhbruhn-cr:R-EU_R0402
- R39: value 1k -> 680R; device rcl:R-EU_R0603 -> jhbruhn-cr:R-EU_R0402
- R4: device rcl:R-EU_R0603 -> jhbruhn-cr:R-EU_R0402
- R40: value 20k -> 1M; device rcl:R-EU_R0603 -> jhbruhn-cr:R-EU_R0402
- R42: device rcl:R-TRIMM64W -> jhbruhn-cr:R-EU_R0402
- R6: value 2k -> 220R; device rcl:R-EU_R0603 -> jhbruhn-cr:R-EU_R0402
- R7: value 120k -> 220R; device rcl:R-EU_R0603 -> jhbruhn-cr:R-EU_R0402
- R8: value 2k -> 56k; device rcl:R-EU_R0603 -> jhbruhn-cr:R-EU_R0402
- T1, T3: value (none) -> 2N3906; device transistor-neu-to92:MMBT3904LT1-NPN-SOT23-BEC -> transistor-neu-to92:MMBT3906LT1-PNP-SOT23-BEC
- T2: value (none) -> BC847BS; device transistor-neu-to92:MMBT3906LT1-PNP-SOT23-BEC -> nxp_60:BC847BS
- T4: value (none) -> 2N3906
- U$1, U$2, U$3, U$4, U$6, U$7, U$8, U$9: device thonkiconn:WQP-PJ301M-12_JACK -> jhbruhn-physical:WQP-PJ301M-12_JACK
- VR1, VR2: device MusicThingModular:9MM_SNAP-IN_POT_ -> jhbruhn-physical:9MM_SNAP-IN_POT_
Connections:
- removed net N$4 (its old number): IC2B.-IN, R1.2, R2.2, R3.2, R6.1
- new net CHANNEL_A: R21.1, SJ1.2, U$4.2
- new net CHANNEL_A_OUT: R50.1, SJ1.1, U$4.3
- new net CHANNEL_B: R44.1, SJ2.2, U$8.2
- new net CHANNEL_B_OUT: R51.1, SJ2.1, U$8.3
- new net N$1: IC2B.+IN, R1.2, R2.1
- new net N$43: C14.1, IC1OTA2.OUT, R38.2, VR3.E
- new net N$44: R40.1, R41.S
- new net N$45: C15.2, R42.2, R43.1, U2B.-IN
- new net N$46: U2B.+IN, VR3.S
- new net N$47: C15.1, R42.1, R44.2, U2B.OUT
- new net N$48: IC4B.-IN, R48.1, R49.2
- new net N$49: T6.B, U2A.-IN, U2A.OUT
- new net N$50: U2A.+IN, VR4.S
- new net N$51: IC1OTA2.I_BIAS, R45.2
- new net N$52: R45.1, R46.2, T6.C
- new net N$53: IC4A.OUT, R49.1, R52.2
- new net N$54: IC4B.OUT, R47.2, R48.2
- new net N$55: IC4A.-IN, R50.2, R51.2, R52.1, R53.2
- new net N$56: SJ3.2, U$1.3
- new net N$57: R53.1, U$2.2
- new net N$58: SJ4.2, U$6.3
- new net REF_10: R54.1, R55.2, SJ3.1, SJ4.1
- net +12V: now also C16.1, C18.1, C20.1, C22.1, C24.+, IC4P.V+, IC5P.V+, R11.2, R18.A, R2.2, R25.2, R34.2, R41.A, R54.2, U1P.V+, U2P.V+; no longer C6.+, R16.1, R24.1, R29.1, R36.1, R4.1, R41.E, R42.E, R9.1, T1.C, T3.C, VR1.E, VR2.E
- net -12V: now also C17.2, C19.2, C21.2, C23.2, C25.-, IC4P.V-, IC5P.V-, R18.E, R23.1, R32.1, R41.E, R46.1, R9.1, U1P.V-, U2P.V-; no longer C7.-, R18.1, R27.1, R38.1, R41.A, R42.A, R7.1, VR1.A, VR2.A
- net GND: now also C16.2, C17.1, C18.2, C19.1, C20.2, C21.1, C22.2, C23.1, C24.-, C25.+, IC2A.+IN, IC2C.+IN, IC2D.+IN, IC4A.+IN, IC4B.+IN, IC5A.+IN, IC5C.+IN, IC5D.+IN, R16.1, R20.2, R37.1, R39.1, R43.2, R55.1, T2-2.B, T2-2.C, T3.E, T5-2.B, T5-2.C, T6.E, VR1.A, VR3.A; no longer C6.-, C7.+, IC1OTA1.IN_N, IC1OTA2.IN_N, R10.2, R17.2, R25.2, R30.2, R34.1, R37.2, R5.2, T2.E, T4.E
- net N$10: now also C10.2, IC1OTA1.IN_N, R15.1, R17.2; no longer IC1BUF1.B, IC1OTA1.OUT, R15.2, R17.1
- net N$11: now also D3.C, IC2A.-IN, R4.2, R5.1, R7.1; no longer IC2A.OUT, R11.2
- net N$12: now also R12.2, T2-1.E, T2-2.E; no longer R12.1, U$3.2
- net N$13: now also C9.1, IC2D.OUT, R12.1, VR2.A; no longer IC1OTA1.IN_P, R12.2, R13.E, R13.S
- net N$14: now also R13.1, U$3.2; no longer R15.1, R41.S
- net N$15: now also IC1OTA1.IN_P, R13.2; no longer R13.A
- net N$16: now also R47.1, U$9.2; no longer R19.2, U$4.2
- net N$17: now also C10.1, IC1OTA1.OUT, R15.2, VR1.E; no longer IC1BUF1.E, R18.2, R19.1
- net N$18: now also R17.1, R18.S; no longer R20.1, U$5.O
- net N$19: now also U1B.+IN, VR1.S; no longer IC1OTA1.I_BIAS, U$5.P
- net N$2: now also C8.2, IC2C.-IN, R10.1, R3.2; no longer R2.1, U$2.2
- net N$20: now also C11.2, R19.2, R20.1, U1B.-IN; no longer R20.2, T2.C
- net N$21: now also IC5B.+IN, R24.2, R25.1; no longer R21.1, U$6.2
- net N$22: now also C11.1, R19.1, R21.2, U1B.OUT; no longer R22.1, U$7.2
- net N$23: now also T3.B, U1A.-IN, U1A.OUT; no longer R23.1, VR2.S
- net N$24: now also U1A.+IN, VR2.S; no longer IC2D.+IN, R21.2, R22.2, R23.2, R26.1
- net N$25: now also IC1OTA1.I_BIAS, R22.2; no longer IC2D.-IN, R24.2, R25.1
- net N$26: now also R22.1, R23.2, T3.C; no longer IC2D.OUT, R26.2, R28.1, T3.B
- net N$27: now also C12.2, IC5C.-IN, R26.2, R33.1; no longer R27.2, T3.E, T4.B
- net N$28: now also IC5B.-IN, IC5B.OUT, R26.1, R27.1; no longer IC2C.+IN, R28.2
- net N$29: now also R24.1, U$6.2; no longer IC2C.-IN, R29.2, R30.1, U$10.S
- net N$3: now also IC2B.-IN, IC2B.OUT, R4.1, R8.1; no longer VR1.S
- net N$30: now also R29.2, R32.2, VR4.E; no longer IC2C.OUT
- net N$31: now also R30.2, T4.E; no longer IC1BUF2.B, IC1OTA2.OUT, R35.2, R36.2, R37.1
- net N$32: now also D4.A, IC5A.OUT, R28.2, R29.1, T4.B, T4.C; no longer R32.1, U$8.2
- net N$33: now also D4.C, IC5A.-IN, R27.2, R28.1, R30.1; no longer IC1OTA2.IN_P, R32.2, R33.E, R33.S
- net N$34: now also C12.1, IC5C.OUT, R33.2, T5-1.B; no longer R33.A, R34.2
- net N$35: now also R35.2, T5-1.E, T5-2.E; no longer R35.1, R42.S
- net N$36: now also C13.2, IC5D.-IN, R34.1, T5-1.C; no longer R39.2, U$9.2
- net N$37: now also C13.1, IC5D.OUT, R35.1, VR4.A; no longer IC1BUF2.E, R38.2, R39.1
- net N$38: now also R36.1, U$7.2; no longer R40.2, T4.C
- net N$39: now also IC1OTA2.IN_P, R36.2, R37.2; no longer R40.1, U$10.O
- net N$40: now also C14.2, IC1OTA2.IN_N, R38.1, R39.2, R40.2; no longer IC1OTA2.I_BIAS, U$10.P
- net N$5: now also C8.1, IC2C.OUT, R10.2, T2-1.B; no longer IC2B.+IN, R4.2, R5.1
- net N$6: now also C9.2, IC2D.-IN, R11.1, T2-1.C; no longer IC2B.OUT, R6.2, R8.1, T1.B
- net N$7: now also R6.2, R9.2, VR2.E; no longer IC2A.-IN, R11.1
- net N$8: no longer T2.B
- net N$9: now also D3.A, IC2A.OUT, R5.2, R6.1, T1.B, T1.C; no longer IC2A.+IN, R10.1, R9.2, U$5.S
Other:
- moved on the sheet: C2, C3, C4, C5, D1, D2, IC1OTA1, IC1OTA2, IC2A, IC2B, IC2C, IC2D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
