File: stereo_mix/hardware_design/pcb/stereo_mix_back_digital.sch (EAGLE design)
At the start: 197 parts, among them IC1 TL072D, IC10 LD117AS50TR, IC2 TL072D, IC3 TL072D, IC4 TL072D, IC5 TL072D, IC6 TL072D, IC7 TL072D, IC8 TL072D, IC9 TL072D, Q1 20MHz, U1 MCP6002_, U10 MCP6002_, U11 MCP4922, U12 MCP4922, U13 ATMEGA328P-AU, U14 TEXAS_INSTRUMENTS_LM4040C5IDB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, U15 TEXAS_INSTRUMENTS_LM4040C10ID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, U16 TEXAS_INSTRUMENTS_LM4040C10ID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, U2 MCP6002_, U3 MCP6002_, U4 MCP6002_, U5 MCP4922, U6 MCP4922, U7 MCP6002_, U8 MCP6002_, U9 MCP6002_

Commit message: Add simulations and schematic for next hardware revision, adding the missing variable bias to the opamp after the MDAC
Parts:
- added C52, C53, C54, C55, C56, C57, C58, C59, C60, C61, C62, C63: 100nF, resistor:C-EUC0402
- added IC11, IC12, IC13, IC14: MCP4822E-SN, dac:MCP4822E-SN
- added IC15, IC16, IC17, IC18: TL072D, linear:TL072D
- added R109, R110, R111, R112, R113, R114, R115, R116: 100k, resistor:R-EU_R0402
- added R117, R118, R119, R120, R121, R122, R123, R124: 43k, resistor:R-EU_R0402
Connections:
- new net BIAS_DAC1_L: IC15A.OUT, R109.2, R29.1
- new net BIAS_DAC1_R: IC15B.OUT, R110.2, R32.1
- new net BIAS_DAC2_L: IC16A.OUT, R111.2, R33.1
- new net BIAS_DAC2_R: IC16B.OUT, R112.2, R36.1
- new net BIAS_DAC3_L: IC17A.OUT, R113.2, R77.1
- new net BIAS_DAC3_R: IC17B.OUT, R114.2, R80.1
- new net BIAS_DAC4_L: IC18A.OUT, R115.2, R81.1
- new net BIAS_DAC4_R: IC18B.OUT, R116.2, R84.1
- new net CS_BIAS_DAC_1: IC11A.CS, U13.PD4(PCINT20/XCK/T0)
- new net CS_BIAS_DAC_2: IC12A.CS, U13.PD5(PCINT21/OC0B/T1)
- new net CS_BIAS_DAC_3: IC13A.CS, U13.PD6(PCINT22/OC0A/AIN0)
- new net CS_BIAS_DAC_4: IC14A.CS, U13.PD7(PCINT23/AIN1)
- new net N$14: IC11A.VOUTA, R117.1
- new net N$16: IC11A.VOUTB, R118.1
- new net N$67: IC12A.VOUTA, R119.1
- new net N$68: IC12A.VOUTB, R120.1
- new net N$70: IC13A.VOUTA, R121.1
- new net N$71: IC13A.VOUTB, R122.1
- new net N$72: IC14A.VOUTA, R123.1
- new net N$73: IC14A.VOUTB, R124.1
- new net N$74: IC15A.-IN, R109.1, R117.2
- new net N$75: IC15B.-IN, R110.1, R118.2
- new net N$76: IC16A.-IN, R111.1, R119.2
- new net N$77: IC16B.-IN, R112.1, R120.2
- new net N$78: IC17A.-IN, R113.1, R121.2
- new net N$79: IC17B.-IN, R114.1, R122.2
- new net N$80: IC18A.-IN, R115.1, R123.2
- new net N$81: IC18B.-IN, R116.1, R124.2
- new net N$84: C52.1, C53.1, C54.1, C55.1, IC11P.VCC, IC12P.VCC, IC13P.VCC, IC14P.VCC
- new net N$85: C52.2, C53.2, C55.2, IC11P.GND, IC12P.GND, IC13P.GND, IC14P.GND
- net +12V: now also C60.1, C61.1, C62.1, C63.1, IC15P.V+, IC16P.V+, IC17P.V+, IC18P.V+
- net -12V: now also C56.2, C57.2, C58.2, C59.2, IC15P.V-, IC16P.V-, IC17P.V-, IC18P.V-
- net AREF_-10: now also U16.ANODE; no longer R29.1, R32.1, R33.1, R36.1, R77.1, R80.1, R81.1, R84.1, U16.CATHODE
- net GND: now also C56.1, C57.1, C58.1, C59.1, C60.2, C61.2, C62.2, C63.2, IC11A.LDAC, IC12A.LDAC, IC13A.LDAC, IC14A.LDAC, IC15A.+IN, IC15B.+IN, IC16A.+IN, IC16B.+IN, IC17A.+IN, IC17B.+IN, IC18A.+IN, IC18B.+IN, U16.CATHODE; no longer U16.ANODE
- net MOSI: now also IC11A.SDI, IC12A.SDI, IC13A.SDI, IC14A.SDI
- net SCK: now also IC11A.SCK, IC12A.SCK, IC13A.SCK, IC14A.SCK
Other:
- moved on the sheet: C22, C24, U16

Commit message: Add new revision of stereo_mix_back hardware, and associated assembly files
Parts:
- removed IC10: LD117AS50TR, v-reg:LD117AS50TR
- removed IC11, IC12, IC13, IC14: MCP4822E-SN, dac:MCP4822E-SN
- removed IC15, IC16, IC17, IC18, IC2, IC3, IC4, IC5, IC6, IC7, IC8, IC9: TL072D, linear:TL072D
- added D3: LM4040AIM3-5.0, jhbruhn-ref:LM4040AIM3-5.0
- added D4, D5: LM4040AIM3-10.0, jhbruhn-ref:LM4040AIM3-10.0
- added U17, U18, U21, U22, U26, U27, U28, U29, U30: TL072AD, jhbruhn-opamp:TL072AD
- added U19, U20, U24, U25: MCP4822E-SN, jhbruhn-dac:MCP4822E-SN
- added U23: ATMEGA328P-AU, jhbruhn-mcu:ATMEGA328P-AU
- C1, C10, C13, C14, C15, C16, C17, C18, C2, C21, C22, C23, C24, C27, C28, C29, C3, C30, C31, C32, C36, C37, C38, C4, C47, C5, C50, C51, C52, C53, C54, C58, C6, C61, C62, C63, C7, C8, C9: device resistor:C-EUC0402 -> jhbruhn-cr:C-EUC0402
- C11, C12, C19, C20: value 100nF -> 4.7nF; device resistor:C-EUC0402 -> jhbruhn-cr:C-EUC0402
- C25, C26: value 18pF -> 100nF; device resistor:C-EUC0402 -> jhbruhn-cr:C-EUC0402
- C33: value EURO_POWER_LOCKFAT-LOCK -> 100nF; device MusicThingModular:EURO_POWER_LOCKFAT-LOCK -> jhbruhn-cr:C-EUC0402
- C34, C35, C45, C46: value 47uF -> 100nF; device rcl:CPOL-EUC -> jhbruhn-cr:C-EUC0402
- C39, C40, C41, C42: value 4.7nF -> 100nF; device resistor:C-EUC0402 -> jhbruhn-cr:C-EUC0402
- C43, C44: value 6.8pF -> 18pF; device resistor:C-EUC0402 -> jhbruhn-cr:C-EUC0402
- C48, C49: value 100nF -> 6.8pF; device resistor:C-EUC0402 -> jhbruhn-cr:C-EUC0402
- C55: value 100nF -> EURO_POWER_LOCKFAT-LOCK; device resistor:C-EUC0402 -> MusicThingModular:EURO_POWER_LOCKFAT-LOCK
- C56, C57, C59, C60: value 100nF -> 47uF; device resistor:C-EUC0402 -> rcl:CPOL-EUC
- IC1: value TL072D -> LD117AS50TR; device linear:TL072D -> v-reg:LD117AS50TR
- R1, R10, R105, R11, R110, R111, R112, R113, R114, R115, R12, R13, R14, R15, R16, R17, R18, R19, R2, R20, R21, R22, R23, R24, R25, R26, R27, R28, R29, R3, R30, R31, R32, R33, R34, R35, R36, R37, R38, R39, R4, R40, R41, R42, R43, R44, R45, R46, R47, R48, R49, R5, R50, R51, R52, R53, R54, R55, R56, R57, R58, R59, R6, R60, R61, R62, R63, R64, R65, R66, R67, R68, R69, R7, R70, R71, R72, R73, R74, R75, R76, R77, R78, R79, R8, R80, R81, R82, R83, R84, R85, R86, R87, R88, R89, R9, R90, R91, R92, R97, R98, R99: device resistor:R-EU_R0402 -> jhbruhn-cr:R-EU_R0402
- R100: value 24k -> 100k; device resistor:R-EU_R0402 -> jhbruhn-cr:R-EU_R0402
- R101: value 24k -> 43k; device resistor:R-EU_R0402 -> jhbruhn-cr:R-EU_R0402
- R102, R103, R104, R94, R95, R96: value 100k -> 43k; device resistor:R-EU_R0402 -> jhbruhn-cr:R-EU_R0402
- R106, R107, R108: value 402R -> 100k; device resistor:R-EU_R0402 -> jhbruhn-cr:R-EU_R0402
- R109: value 100k -> 10k; device resistor:R-EU_R0402 -> jhbruhn-cr:R-EU_R0402
- R116: value 100k -> 24k; device resistor:R-EU_R0402 -> jhbruhn-cr:R-EU_R0402
- R117: value 43k -> 24k; device resistor:R-EU_R0402 -> jhbruhn-cr:R-EU_R0402
- R118, R119, R120, R121: value 43k -> 100k; device resistor:R-EU_R0402 -> jhbruhn-cr:R-EU_R0402
- R122, R123, R124: value 43k -> 470R; device resistor:R-EU_R0402 -> jhbruhn-cr:R-EU_R0402
- R93: value 10k -> 43k; device resistor:R-EU_R0402 -> jhbruhn-cr:R-EU_R0402
- U1, U10, U8, U9: value MCP6002_ -> TL072AD; device MusicThingModular:MCP6002_ -> jhbruhn-opamp:TL072AD
- U11, U12, U5: value MCP4922 -> MCP6002E/SN; device MCP4922:MCP4922 -> jhbruhn-opamp:MCP6002E/SN
- U13: value ATMEGA328P-AU -> MCP6002E/SN; device Microcontroller:ATMEGA328P-AU -> jhbruhn-opamp:MCP6002E/SN
- U14: value TEXAS_INSTRUMENTS_LM4040C5IDBZR -> MCP6002E/SN; device lm4040:TEXAS_INSTRUMENTS_LM4040C5IDBZR -> jhbruhn-opamp:MCP6002E/SN
- U15, U16: value TEXAS_INSTRUMENTS_LM4040C10IDBZR -> MCP4922E/SL; device lm4040:TEXAS_INSTRUMENTS_LM4040C10IDBZR -> jhbruhn-dac:MCP4922E/SL
- U2, U3, U4: value MCP6002_ -> MCP6002E/SN; device MusicThingModular:MCP6002_ -> jhbruhn-opamp:MCP6002E/SN
- U6: value MCP4922 -> MCP4922E/SL; device MCP4922:MCP4922 -> jhbruhn-dac:MCP4922E/SL
- U7: value MCP6002_ -> MCP4922E/SL; device MusicThingModular:MCP6002_ -> jhbruhn-dac:MCP4922E/SL
Connections:
- removed net 3_CV_PAN_IN: R43.1, R44.1
- removed net N$84: C52.1, C53.1, C54.1, C55.1, IC11P.VCC, IC12P.VCC, IC13P.VCC, IC14P.VCC
- removed net N$85: C52.2, C53.2, C55.2, IC11P.GND, IC12P.GND, IC13P.GND, IC14P.GND
- net +12V: now also C13.1, C41.1, C42.1, C45.1, C46.1, C52.1, C53.1, C54.1, C56.+, C59.+, IC1.IN, R122.2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; no longer C11.1, C30.1, C31.1, C32.1, C34.+, C45.+, C60.1, C61.1, C62.1, C63.1, IC10.IN, IC15P.V+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
- net +5V: now also C24.1, C25.1, C26.1, C27.1, C28.1, C29.1, C30.1, C31.1, C32.1, C33.1, C35.1, C36.1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; no longer C13.1, C14.1, C19.1, C20.1, C46.+, C47.1, C48.1, C49.1, C50.1, C51.1, IC10.OUT, R93.2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
- net -12V: now also C14.2, C37.2, C38.2, C39.2, C40.2, C47.2, C50.2, C51.2, C57.-, R124.2, U10P.V-, U17P.V-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; no longer C12.2, C27.2, C28.2, C29.2, C35.-, C56.2, C57.2, C58.2, C59.2, IC15P.V-, IC16P.V-, IC17P.V-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
- net 1_PAN_ATT_W: now also U1A.+IN; no longer IC1A.+IN
- net 2_PAN_ATT_W: now also U1B.+IN; no longer IC1B.+IN
- net 3_PAN_ATT_W: now also U10A.+IN; no longer IC4A.+IN
- net 3_PAN_CV_IN: now also R43.1, R44.1
- net 4_PAN_ATT_W: now also U10B.+IN; no longer IC4B.+IN
- net AREF_-10: now also C63.1, D5.A, R124.1; no longer C38.1, R108.1, U16.ANODE
- net AUX_IN_L: now also R110.1; no longer R94.1
- net AUX_IN_R: now also R111.1; no longer R95.1
- net BAL_N_L: now also R120.2, U29B.OUT; no longer IC8B.OUT, R104.2
- net BAL_N_R: now also R121.2, U30B.OUT; no longer IC9B.OUT, R105.2
- net BAL_P_L: now also R116.2, R118.1, U29A.OUT; no longer IC8A.OUT, R100.2, R102.1
- net BAL_P_R: now also R117.2, R119.1, U30A.OUT; no longer IC9A.OUT, R101.2, R103.1
- net BIAS_DAC1_L: now also R97.2, U21A.OUT; no longer IC15A.OUT, R109.2
- net BIAS_DAC1_R: now also R98.2, U21B.OUT; no longer IC15B.OUT, R110.2
- net BIAS_DAC2_L: now also R99.2, U22A.OUT; no longer IC16A.OUT, R111.2
- net BIAS_DAC2_R: now also R100.2, U22B.OUT; no longer IC16B.OUT, R112.2
- net BIAS_DAC3_L: now also R105.2, U26A.OUT; no longer IC17A.OUT, R113.2
- net BIAS_DAC3_R: now also R106.2, U26B.OUT; no longer IC17B.OUT, R114.2
- net BIAS_DAC4_L: now also R107.2, U27A.OUT; no longer IC18A.OUT, R115.2
- net BIAS_DAC4_R: now also R108.2, U27B.OUT; no longer IC18B.OUT, R116.2
- net BYPASS_L: now also C48.2, R112.2, U28A.OUT; no longer C43.2, IC7A.OUT, R96.2
- net BYPASS_R: now also C49.2, R113.2, U28B.OUT; no longer C44.2, IC7B.OUT, R97.2
- net CS_BIAS_DAC_1: now also U19A.CS, U23.PD4(PCINT20/XCK/T0); no longer IC11A.CS, U13.PD4(PCINT20/XCK/T0)
- net CS_BIAS_DAC_2: now also U20A.CS, U23.PD5(PCINT21/OC0B/T1); no longer IC12A.CS, U13.PD5(PCINT21/OC0B/T1)
- net CS_BIAS_DAC_3: now also U23.PD6(PCINT22/OC0A/AIN0), U24A.CS; no longer IC13A.CS, U13.PD6(PCINT22/OC0A/AIN0)
- net CS_BIAS_DAC_4: now also U23.PD7(PCINT23/AIN1), U25A.CS; no longer IC14A.CS, U13.PD7(PCINT23/AIN1)
- net CS_DAC_1: now also U23.PD0(RXD/PCINT16), U6.!CS; no longer U13.PD0(RXD/PCINT16), U5.!CS
- net CS_DAC_2: now also U23.PD1(TXD/PCINT17), U7.!CS; no longer U13.PD1(TXD/PCINT17), U6.!CS
- net CS_DAC_3: now also U15.!CS, U23.PD2(INT0/PCINT18); no longer U11.!CS, U13.PD2(INT0/PCINT18)
- net CS_DAC_4: now also U16.!CS, U23.PD3(PCINT19/OC2B/INT1); no longer U12.!CS, U13.PD3(PCINT19/OC2B/INT1)
- net GND: now also C14.1, C27.2, C28.2, C29.2, C33.2, C34.2, C35.2, C37.1, C38.1, C39.1, C40.1, C41.2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; no longer C11.2, C12.1, C14.2, C19.2, C20.2, C27.1, C28.1, C29.1, C33.GND, C34.-, C35.+, C37.2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
- net MISO: now also U23.(PCINT4/MISO)PB4; no longer U13.(PCINT4/MISO)PB4
- net MOSI: now also U15.SDI, U16.SDI, U19A.SDI, U20A.SDI, U23.(PCINT3/OC2A/MOSI)PB3, U24A.SDI, U25A.SDI, U7.SDI; no longer IC11A.SDI, IC12A.SDI, IC13A.SDI, IC14A.SDI, U11.SDI, U12.SDI, U13.(PCINT3/OC2A/MOSI)PB3, U5.SDI
- net N$1: now also U6.VOUT_A; no longer U5.VOUT_A
- net N$10: now also U6.VOUT_B; no longer U5.VOUT_B
- net N$11: now also C43.1, U23.(PCINT7/XTAL2/TOSC2)PB7; no longer C25.1, U13.(PCINT7/XTAL2/TOSC2)PB7
- net N$12: now also C11.1, U4A.-IN; no longer C39.1, U3A.-IN
- net N$13: now also U1A.OUT; no longer IC1A.OUT
- net N$14: now also R93.1, U19A.VOUTA; no longer IC11A.VOUTA, R117.1
- net N$15: now also U5A.+IN; no longer U4A.+IN
- net N$16: now also R94.1, U19A.VOUTB; no longer IC11A.VOUTB, R118.1
- net N$17: now also U5B.+IN; no longer U4B.+IN
- net N$18: now also U1A.-IN; no longer IC1A.-IN
- net N$19: now also U3B.-IN; no longer U2B.-IN
- net N$2: now also U2B.-IN; no longer U1B.-IN
- net N$20: now also U3B.OUT, U7.VREFB; no longer U2B.OUT, U6.VREFB
- net N$21: now also U3A.OUT, U7.VREFA; no longer U2A.OUT, U6.VREFA
- net N$22: now also U3A.-IN; no longer U2A.-IN
- net N$23: now also U7.VOUT_A; no longer U6.VOUT_A
- net N$24: now also U9A.-IN; no longer IC3A.-IN
- net N$25: now also U9A.OUT; no longer IC3A.OUT
- net N$26: now also U9B.-IN; no longer IC3B.-IN
- net N$27: now also U7.VOUT_B; no longer U6.VOUT_B
- net N$28: now also U9B.OUT; no longer IC3B.OUT
- net N$29: now also U11B.-IN; no longer U7B.-IN
- net N$3: now also U8A.-IN; no longer IC2A.-IN
- net N$30: now also U11B.OUT, U15.VREFB; no longer U11.VREFB, U7B.OUT
- net N$31: now also U11A.OUT, U15.VREFA; no longer U11.VREFA, U7A.OUT
- net N$32: now also R114.1, R116.1, U29A.-IN; no longer IC8A.-IN, R100.1, R98.1
- net N$33: now also U11A.-IN; no longer U7A.-IN
- net N$34: now also U15.VOUT_A; no longer U11.VOUT_A
- net N$35: now also U17A.-IN; no longer IC5A.-IN
- net N$36: now also U17A.OUT; no longer IC5A.OUT
- net N$37: now also U17B.-IN; no longer IC5B.-IN
- net N$38: now also U15.VOUT_B; no longer U11.VOUT_B
- net N$39: now also U17B.OUT; no longer IC5B.OUT
- net N$4: now also U2A.OUT, U6.VREFA; no longer U1A.OUT, U5.VREFA
- net N$40: now also U12B.-IN; no longer U8B.-IN
- net N$41: now also U12B.OUT, U16.VREFB; no longer U12.VREFB, U8B.OUT
- net N$42: now also C12.1, U4B.-IN; no longer C40.1, U3B.-IN
- net N$43: now also R119.2, R121.1, U30B.-IN; no longer IC9B.-IN, R103.2, R105.1
- net N$44: now also U12A.OUT, U16.VREFA; no longer U12.VREFA, U8A.OUT
- net N$45: now also R118.2, R120.1, U29B.-IN; no longer IC8B.-IN, R102.2, R104.1
- net N$46: now also U12A.-IN; no longer U8A.-IN
- net N$47: now also C55.+12V; no longer C33.+12V
- net N$48: now also C55.-12V; no longer C33.-12V
- net N$49: now also U16.VOUT_A; no longer U12.VOUT_A
- net N$5: now also U2B.OUT, U6.VREFB; no longer U1B.OUT, U5.VREFB
- net N$50: now also U18A.-IN; no longer IC6A.-IN
- net N$51: now also U18A.OUT; no longer IC6A.OUT
- net N$52: now also U18B.-IN; no longer IC6B.-IN
- net N$53: now also U16.VOUT_B; no longer U12.VOUT_B
- net N$54: now also U18B.OUT; no longer IC6B.OUT
- net N$55: now also R115.1, R117.1, U30A.-IN; no longer IC9A.-IN, R101.1, R99.1
- net N$56: now also U1B.OUT; no longer IC1B.OUT
- net N$57: now also U1B.-IN; no longer IC1B.-IN
- net N$58: now also C34.1, U23.AREF; no longer C24.1, U13.AREF
- net N$59: now also C19.1, U14A.-IN; no longer C41.1, U10A.-IN
- net N$6: now also U2A.-IN; no longer U1A.-IN
- net N$60: now also U10A.OUT; no longer IC4A.OUT
- net N$61: now also U10A.-IN; no longer IC4A.-IN
- net N$62: now also C44.1, U23.(PCINT6/XTAL1/TOSC1)PB6; no longer C26.1, U13.(PCINT6/XTAL1/TOSC1)PB6
- net N$63: now also C20.1, U14B.-IN; no longer C42.1, U10B.-IN
- net N$64: now also U10B.OUT; no longer IC4B.OUT
- net N$65: now also U10B.-IN; no longer IC4B.-IN
- net N$66: now also U13A.+IN; no longer U9A.+IN
- net N$67: now also R95.1, U20A.VOUTA; no longer IC12A.VOUTA, R119.1
- net N$68: now also R96.1, U20A.VOUTB; no longer IC12A.VOUTB, R120.1
- net N$69: now also U13B.+IN; no longer U9B.+IN
- net N$7: now also U8B.OUT; no longer IC2B.OUT
- net N$70: now also R101.1, U24A.VOUTA; no longer IC13A.VOUTA, R121.1
- net N$71: now also R102.1, U24A.VOUTB; no longer IC13A.VOUTB, R122.1
- net N$72: now also R103.1, U25A.VOUTA; no longer IC14A.VOUTA, R123.1
- net N$73: now also R104.1, U25A.VOUTB; no longer IC14A.VOUTB, R124.1
- net N$74: now also R93.2, R97.1, U21A.-IN; no longer IC15A.-IN, R109.1, R117.2
- net N$75: now also R94.2, R98.1, U21B.-IN; no longer IC15B.-IN, R110.1, R118.2
- net N$76: now also R95.2, R99.1, U22A.-IN; no longer IC16A.-IN, R111.1, R119.2
- net N$77: now also R100.1, R96.2, U22B.-IN; no longer IC16B.-IN, R112.1, R120.2
- net N$78: now also R101.2, R105.1, U26A.-IN; no longer IC17A.-IN, R113.1, R121.2
- net N$79: now also R102.2, R106.1, U26B.-IN; no longer IC17B.-IN, R114.1, R122.2
- net N$8: now also U8A.OUT; no longer IC2A.OUT
- net N$80: now also R103.2, R107.1, U27A.-IN; no longer IC18A.-IN, R115.1, R123.2
- net N$81: now also R104.2, R108.1, U27B.-IN; no longer IC18B.-IN, R116.1, R124.2
- net N$9: now also U8B.-IN; no longer IC2B.-IN
- net OUT_L: now also R114.2; no longer R98.2
- net OUT_R: now also R115.2; no longer R99.2
- net PAN_CV_1: now also C11.2, U23.(ADC4/SDA/PCINT12)PC4, U4A.OUT; no longer C39.2, U13.(ADC4/SDA/PCINT12)PC4, U3A.OUT
- net PAN_CV_2: now also C12.2, U23.(ADC5/SCL/PCINT13)PC5, U4B.OUT; no longer C40.2, U13.(ADC5/SCL/PCINT13)PC5, U3B.OUT
- net PAN_CV_3: now also C19.2, U14A.OUT, U23.ADC6; no longer C41.2, U10A.OUT, U13.ADC6
- net PAN_CV_4: now also C20.2, U14B.OUT, U23.ADC7; no longer C42.2, U10B.OUT, U13.ADC7
- net REF_10: now also C61.1, D4.C, R123.1; no longer C37.1, R107.1, U15.CATHODE
- net REF_5: now also C58.1, D3.C, R122.1; no longer C36.1, R106.1, U14.CATHODE
- net RESET: now also R109.1, U23.(RESET/PCINT14)PC6; no longer R93.1, U13.(RESET/PCINT14)PC6
- net SCK: now also U15.SCK, U16.SCK, U19A.SCK, U20A.SCK, U23.(SCK/PCINT5)PB5, U24A.SCK, U25A.SCK, U7.SCK; no longer IC11A.SCK, IC12A.SCK, IC13A.SCK, IC14A.SCK, U11.SCK, U12.SCK, U13.(SCK/PCINT5)PB5, U5.SCK
- net SUM_L: now also C48.1, R110.2, R112.1, U28A.-IN; no longer C43.1, IC7A.-IN, R94.2, R96.1
- net SUM_R: now also C49.1, R111.2, R113.1, U28B.-IN; no longer C44.1, IC7B.-IN, R95.2, R97.1
- net VOL_CV_1: now also U23.(ADC0/PCINT8)PC0, U5A.-IN, U5A.OUT; no longer U13.(ADC0/PCINT8)PC0, U4A.-IN, U4A.OUT
- net VOL_CV_2: now also U23.(ADC1/PCINT9)PC1, U5B.-IN, U5B.OUT; no longer U13.(ADC1/PCINT9)PC1, U4B.-IN, U4B.OUT
- net VOL_CV_3: now also U13A.-IN, U13A.OUT, U23.(ADC2/PCINT10)PC2; no longer U13.(ADC2/PCINT10)PC2, U9A.-IN, U9A.OUT
- net VOL_CV_4: now also U13B.-IN, U13B.OUT, U23.(ADC3/PCINT11)PC3; no longer U13.(ADC3/PCINT11)PC3, U9B.-IN, U9B.OUT

Commit message: Start revamp of stereo mix pcb
Parts:
- removed C43, C44: 18pF, jhbruhn-cr:C-EUC0402
- removed JP1: (no value), pinhead:PINHD-1X20
- removed JP2: (no value), pinhead:PINHD-1X9
- removed JP4, JP6, JP7: (no value), jumper:JP2E
- removed JP5: (no value), pinhead:PINHD-1X5
- removed Q1: 20MHz, crystal:CRYSTALHC49UP
- removed R115, R118, R119, R120, R121, R44, R46, R49, R50, R6: 100k, jhbruhn-cr:R-EU_R0402
- removed R116, R117: 24k, jhbruhn-cr:R-EU_R0402
- removed U29, U30: TL072AD, jhbruhn-opamp:TL072AD
- added J1, J10, J11, J12, J13, J14, J15, J16, J17, J18, J2, J3, J4, J5, J6, J7, J8, J9: WQP-PJ301M-12_JACK, jhbruhn-physical:WQP-PJ301M-12_JACK
- added VR1, VR2, VR3, VR4, VR5, VR6, VR7, VR8: (no value), jhbruhn-physical:9MM_SNAP-IN_POT_
- C56, C57, C59, C60: device rcl:CPOL-EUC -> rcl:CPOL-EUA/3216-18W
Connections:
- removed net 1_PAN_ATT_W: JP1.5, R2.2, R5.2, U1A.+IN
- removed net 2_PAN_ATT_W: JP1.11, R4.2, R6.2, U1B.+IN
- removed net 3_PAN_ATT_W: JP1.17, R44.2, R49.2, U10A.+IN
- removed net 4_PAN_ATT_W: JP2.5, R46.2, R50.2, U10B.+IN
- removed net BAL_N_L: JP6.2, R120.2, U29B.OUT
- removed net BAL_N_R: JP7.2, R121.2, U30B.OUT
- removed net BAL_P_L: JP6.1, R116.2, R118.1, U29A.OUT
- removed net BAL_P_R: JP7.1, R117.2, R119.1, U30A.OUT
- removed net BYPASS_L: C48.2, JP4.1, JP5.3, R112.2, U28A.OUT
- removed net BYPASS_R: C49.2, JP4.2, JP5.4, R113.2, U28B.OUT
- removed net N$42: C12.1, R23.2, R24.2, R27.1, U4B.-IN
- removed net N$62: C44.1, Q1.1, U23.(PCINT6/XTAL1/TOSC1)PB6
- removed net N$63: C20.1, R71.2, R72.2, R74.1, U14B.-IN
- new net N$83: U10A.+IN, VR6.S
- net +12V: no longer JP1.1, U29P.V+, U30P.V+
- net -12V: no longer JP1.19, U29P.V-, U30P.V-
- net 1_IN_L: now also J1.2; no longer JP1.2
- net 1_IN_R: now also J2.2; no longer JP1.3
- net 1_PAN_CV_IN: now also J10.2, R114.1; no longer JP1.4, R1.1, R2.1
- net 1_VOLUME_CV: now also J9.2; no longer JP1.7
- net 2_IN_L: now also J3.2; no longer JP1.8
- net 2_IN_R: now also J4.2; no longer JP1.9
- net 2_PAN_CV_IN: now also J12.2, R2.1; no longer JP1.10, R3.1, R4.1
- net 2_VOLUME_CV: now also J11.2; no longer JP1.13
- net 3_IN_L: now also J5.2; no longer JP1.14
- net 3_IN_R: now also J6.2; no longer JP1.15
- net 3_PAN_CV_IN: now also J14.2, R4.1; no longer JP1.16, R43.1, R44.1
- net 3_VOLUME_CV: now also J13.2; no longer JP2.1
- net 4_IN_L: now also J7.2; no longer JP2.2
- net 4_IN_R: now also J8.2; no longer JP2.3
- net 4_PAN_CV_IN: now also J16.2, R5.1; no longer JP2.4, R45.1, R46.1
- net 4_VOLUME_CV: now also J15.2; no longer JP2.7
- net GND: now also U13A.+IN, U5A.+IN, VR2.A, VR4.A, VR6.A, VR8.A; no longer C43.2, C44.2, JP1.12, JP1.18, JP1.20, JP1.6, JP2.6, JP4.3, JP5.5, JP6.3, JP7.3, R49.1, R5.1, R50.1, R6.1, U14B.+IN, U29A.+IN, U29B.+IN, U30A.+IN, U30B.+IN, U4B.+IN
- net N$11: now also C12.1, R2.2, R23.2, R24.2, R27.1, U5A.-IN; no longer C43.1, Q1.2, U23.(PCINT7/XTAL2/TOSC2)PB7
- net N$12: now also U1A.+IN, VR2.S; no longer C11.1, R21.2, R22.2, R26.1, U4A.-IN
- net N$15: now also U4B.+IN; no longer U5A.+IN
- net N$32: now also C11.1, R114.2, R21.2, R22.2, R26.1, U4A.-IN; no longer R114.1, R116.1, U29A.-IN
- net N$43: now also U1B.+IN, VR4.S; no longer R119.2, R121.1, U30B.-IN
- net N$45: now also U10B.+IN, VR8.S; no longer R118.2, R120.1, U29B.-IN
- net N$55: now also C20.1, R5.2, R71.2, R72.2, R74.1, U13A.-IN; no longer R115.1, R117.1, U30A.-IN
- net N$59: now also R4.2
- net N$66: now also U14B.+IN; no longer U13A.+IN
- net OUT_L: now also C48.2, J17.2, R112.2, U28A.OUT; no longer JP5.1, R114.2
- net OUT_R: now also C49.2, J18.2, R113.2, U28B.OUT; no longer JP5.2, R115.2
- net PAN_CV_2: now also U5A.OUT; no longer U4B.OUT
- net PAN_CV_4: now also U13A.OUT; no longer U14B.OUT
- net REF_10: no longer JP2.9
- net REF_5: now also R1.1, R3.1, R43.1, R45.1, VR2.E, VR4.E, VR6.E, VR8.E; no longer JP2.8
- net VOL_CV_1: now also U4B.-IN, U4B.OUT; no longer U5A.-IN, U5A.OUT
- net VOL_CV_3: now also U14B.-IN, U14B.OUT; no longer U13A.-IN, U13A.OUT
Other:
- moved on the sheet: R1, R2, R3, R4, R43, R45, R5, U13A, U14B, U4B, U5A

Commit message: Add new hardware revision of stereo mix
Parts:
- removed C45, C46, C47, C50, C51, C52, C53, C54, C58, C61, C62, C63: 100nF, jhbruhn-cr:C-EUC0402
- removed C48, C49: 6.8pF, jhbruhn-cr:C-EUC0402
- removed C55: EURO_POWER_LOCKFAT-LOCK, MusicThingModular:EURO_POWER_LOCKFAT-LOCK
- removed C56, C57, C59, C60: 47uF, rcl:CPOL-EUA/3216-18W
- removed D4, D5: LM4040AIM3-10.0, jhbruhn-ref:LM4040AIM3-10.0
- removed ISP1: AVRISP-6, adafruit:AVRISP-6
- removed JP3: (no value), jumper:JP2E
- removed R100, R105, R106, R107, R108, R110, R111, R112, R113, R114, R91, R92, R97, R98, R99: 100k, jhbruhn-cr:R-EU_R0402
- removed R101, R102, R103, R104, R93, R94, R95, R96: 43k, jhbruhn-cr:R-EU_R0402
- removed R109: 10k, jhbruhn-cr:R-EU_R0402
- removed R122, R123, R124: 470R, jhbruhn-cr:R-EU_R0402
- removed U23: ATMEGA328P-AU, jhbruhn-mcu:ATMEGA328P-AU
- removed U24, U25: MCP4822E-SN, jhbruhn-dac:MCP4822E-SN
- removed U26, U27, U28: TL072AD, jhbruhn-opamp:TL072AD
- added IC2: AMS1117-3.3, jhbruhn-ic:AMS1117-3.3
- added J19: WQP-PJ301M-12_JACK, jhbruhn-physical:WQP-PJ301M-12_JACK
- added JP1, JP2: (no value), jumper:JP2E
- added R44: 15k, jhbruhn-cr:R-EU_R0402
- added R46, R49, R50: 47k, jhbruhn-cr:R-EU_R0402
- added R6: 100k, jhbruhn-cr:R-EU_R0402
- added X1: 8MHz, jhbruhn-cdr:XTALNX5032
- C11, C12: value 4.7nF -> 100nF
- C21, C22: value 100nF -> 4.7nF
- C26, C27: value 100nF -> 22pF
- C32, C33: value 100nF -> 6.8pF
- C36: value 100nF -> EURO_POWER_LOCKFAT-LOCK; device jhbruhn-cr:C-EUC0402 -> MusicThingModular:EURO_POWER_LOCKFAT-LOCK
- C37, C38, C39, C41: value 100nF -> 10uF; device jhbruhn-cr:C-EUC0402 -> jhbruhn-cdr:CPOL-EUA/3216-18R
- D1, D2: value 1N4001 -> 1N4148W; device adafruit:DIODESMA -> jhbruhn-cdr:DIODE-SOD123
- D3: value LM4040AIM3-5.0 -> LM4040AIM3-10.0; device jhbruhn-ref:LM4040AIM3-5.0 -> jhbruhn-ref:LM4040AIM3-10.0
- IC1: value LD117AS50TR -> 4051D; device v-reg:LD117AS50TR -> jhbruhn-ic:4051D
- J17: value WQP-PJ301M-12_JACK -> CORTEX_DEBUG_PTH; device jhbruhn-physical:WQP-PJ301M-12_JACK -> jhbruhn-physical:CORTEX_DEBUG_PTH
- R1, R3, R33, R37, R39, R5, R7: value 100k -> 91k
- R10, R11, R12, R41, R42, R43, R9: value 100k -> 15k
- R13, R14, R15, R16, R45, R47, R48, R51, R52: value 100k -> 47k
- R17, R18, R19, R20: value 24k -> 47k
- R21: value 200k -> 100k
- R23: value 200k -> 300k
- R25, R28, R57, R58, R59, R60: value 100k -> 300k
- R26: value 51k -> 300k
- R27: value 51k -> 100k
- R30, R31, R34, R66, R68, R82, R83: value 24k -> 100k
- R35: value 24k -> 91k
- R65, R67, R78, R79: value 24k -> 200k
- R73, R74: value 51k -> 33k
- R75, R76: value 100k -> 33k
- R77, R80: value 100k -> 200k
- R85: value 100k -> 10k
- R90: value 100k -> 470R
- U1, U10, U9: value TL072AD -> MCP4822E-SN; device jhbruhn-opamp:TL072AD -> jhbruhn-dac:MCP4822E-SN
- U11, U12, U3, U4: value MCP6002E/SN -> MCP6002T-I/SN; device jhbruhn-opamp:MCP6002E/SN -> jhbruhn-opamp:MCP6002T-I/SN
- U13, U14, U5: value MCP6002E/SN -> MCP4922E/SL; device jhbruhn-opamp:MCP6002E/SN -> jhbruhn-dac:MCP4922E/SL
- U15, U16, U7: value MCP4922E/SL -> TL072CD; device jhbruhn-dac:MCP4922E/SL -> jhbruhn-opamp:TL072CD
- U17, U18: value TL072AD -> MCP6002T-I/SN; device jhbruhn-opamp:TL072AD -> jhbruhn-opamp:MCP6002T-I/SN
- U19, U20: value MCP4822E-SN -> MCP6002T-I/SN; device jhbruhn-dac:MCP4822E-SN -> jhbruhn-opamp:MCP6002T-I/SN
- U2: value MCP6002E/SN -> MCP4822E-SN; device jhbruhn-opamp:MCP6002E/SN -> jhbruhn-dac:MCP4822E-SN
- U21: value TL072AD -> STM32F030C8T6; device jhbruhn-opamp:TL072AD -> jhbruhn-mcu:STM32F030C8T6
- U22, U8: value TL072AD -> TL072CD; device jhbruhn-opamp:TL072AD -> jhbruhn-opamp:TL072CD
Connections:
- removed net 1_PAN_CV_IN: J10.2, R114.1
- removed net 1_VOLUME_CV: J9.2, R25.2
- removed net N$12: U1A.+IN, VR2.S
- removed net N$13: R22.1, R7.2, U1A.OUT
- removed net N$18: R1.2, R7.1, U1A.-IN
- removed net N$43: U1B.+IN, VR4.S
- removed net N$45: U10B.+IN, VR8.S
- removed net N$56: R24.1, R8.2, U1B.OUT
- removed net N$57: R3.2, R8.1, U1B.-IN
- removed net N$58: C34.1, U23.AREF
- removed net N$60: R53.2, R70.1, U10A.OUT
- removed net N$61: R43.2, R53.1, U10A.-IN
- removed net N$64: R54.2, R72.1, U10B.OUT
- removed net N$65: R45.2, R54.1, U10B.-IN
- removed net N$74: R93.2, R97.1, U21A.-IN
- removed net N$77: R100.1, R96.2, U22B.-IN
- removed net N$78: R101.2, R105.1, U26A.-IN
- removed net N$79: R102.2, R106.1, U26B.-IN
- removed net N$80: R103.2, R107.1, U27A.-IN
- removed net N$81: R104.2, R108.1, U27B.-IN
- removed net N$83: U10A.+IN, VR6.S
- removed net REF_10: C61.1, D4.C, R123.1
- removed net REF_5: C58.1, D3.C, R1.1, R122.1, R3.1, R43.1, R45.1, VR2.E, VR4.E, VR6.E, VR8.E
- removed net RESET: ISP1.RST, R109.1, U23.(RESET/PCINT14)PC6
- new net +3V3: C10.1, C11.1, C12.1, C13.1, C14.1, C15.1, C16.1, C17.1, C18.1, C23.1, C24.1, C25.1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
- new net MUX_ADDR_0: IC1A.A, U21.PB12/SPI2_NSS/TIM1_BKIN/EVENTOUT
- new net MUX_ADDR_1: IC1A.B, U21.PB13/SPI2_SCK/TIM1_CH1N
- new net MUX_ADDR_2: IC1A.C, U21.PB14/SPI2_MISO/TIM1_CH2N/TIM15_CH1
- new net N$84: J9.2, R66.1
- new net N$89: J13.2, R77.2
- new net NRST: J17.!RESET, R85.1, U21.NRST
- new net PAN_1_POT: IC1A.X4, VR3.S
- new net PAN_2_POT: IC1A.X5, VR7.S
- new net PAN_3_POT: IC1A.X6, VR4.S
- new net PAN_4_POT: IC1A.X7, VR8.S
- new net POT_MUX: IC1A.X, U21.PB0/TIM3_CH3/TIM1_CH2N/EVENTOUT/ADC_IN8
- new net SWDCLK: J17.SWDCLK/TCK, U21.PA14/USART2_TX/SWCLK
- new net SWDIO: J17.SWDIO/TMS, U21.PA13/IR_OUT/SWDIO
- new net VOL_1_POT: IC1A.X0, VR1.S
- new net VOL_2_POT: IC1A.X1, VR5.S
- new net VOL_3_POT: IC1A.X2, VR2.S
- new net VOL_4_POT: IC1A.X3, VR6.S
- net +12V: now also C35.1, C37.+, C39.+, IC2.IN, U15P.V+, U16P.V+, U7P.V+; no longer C13.1, C41.1, C42.1, C45.1, C46.1, C52.1, C53.1, C54.1, C56.+, C59.+, C9.1, IC1.IN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
- net +5V: now also U13.!SHDN, U13.VDD, U14.!SHDN, U14.VDD, U5.!SHDN, U5.VDD; no longer C15.1, C16.1, C17.1, C18.1, C21.1, C22.1, C23.1, C24.1, C25.1, C26.1, C27.1, C28.1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
- net -12V: now also C34.2, C38.-, R90.2, U15P.V-, U16P.V-, U7P.V-; no longer C10.2, C14.2, C37.2, C38.2, C39.2, C40.2, C47.2, C50.2, C51.2, C57.-, R124.2, U10P.V-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
- net 1_IN_L: now also R2.1; no longer R10.1
- net 1_IN_R: now also R4.1; no longer R12.1
- net 2_IN_L: now also R6.1; no longer R14.1
- net 2_IN_R: now also R8.1; no longer R16.1
- net 2_PAN_CV_IN: now also J10.2, R68.1; no longer J12.2, R2.1
- net 2_VOLUME_CV: now also J14.2, R78.2; no longer J11.2, R37.2
- net 3_IN_L: now also R34.1; no longer R56.1
- net 3_IN_R: now also R36.1; no longer R58.1
- net 3_PAN_CV_IN: now also J11.2, R70.1; no longer J14.2, R4.1
- net 3_VOLUME_CV: now also J15.2, R79.2; no longer J13.2, R63.2
- net 4_IN_L: now also R38.1; no longer R60.1
- net 4_IN_R: now also R40.1; no longer R62.1
- net 4_PAN_CV_IN: now also J12.2, R72.1; no longer J16.2, R5.1
- net 4_VOLUME_CV: now also J16.2, R80.2; no longer J15.2, R75.2
- net AREF_-10: now also C40.1, D3.A, R1.1, R3.1, R33.1, R35.1, R37.1, R39.1, R5.1, R65.1, R67.1, R7.1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; no longer C63.1, D5.A, R11.1, R124.1, R13.1, R15.1, R21.1, R23.1, R55.1, R57.1, R59.1, R61.1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
- net AUX_IN_L: now also JP1.1, R86.1; no longer JP3.1, R110.1
- net AUX_IN_R: now also JP1.2, R87.1; no longer JP3.2, R111.1
- net BIAS_DAC1_L: now also R16.1, U1A.VOUTA; no longer R29.1, R97.2, U21A.OUT
- net BIAS_DAC1_R: now also R15.1, U1A.VOUTB; no longer R32.1, R98.2, U21B.OUT
- net BIAS_DAC2_L: now also R20.1, U2A.VOUTA; no longer R33.1, R99.2, U22A.OUT
- net BIAS_DAC2_R: now also R19.1, U2A.VOUTB; no longer R100.2, R36.1, U22B.OUT
- net BIAS_DAC3_L: now also R51.1, U9A.VOUTA; no longer R105.2, R77.1, U26A.OUT
- net BIAS_DAC3_R: now also R47.1, U9A.VOUTB; no longer R106.2, R80.1, U26B.OUT
- net BIAS_DAC4_L: now also R52.1, U10A.VOUTA; no longer R107.2, R81.1, U27A.OUT
- net BIAS_DAC4_R: now also R50.1, U10A.VOUTB; no longer R108.2, R84.1, U27B.OUT
- net CS_BIAS_DAC_1: now also U1A.CS, U21.PB8/I2C1_SCL/TIM16_CH1; no longer U19A.CS, U23.PD4(PCINT20/XCK/T0)
- net CS_BIAS_DAC_2: now also U21.PB9/I2C1_SDA/IR_OUT/SPI2_NSS/TIM17_CH1/EVENTOUT, U2A.CS; no longer U20A.CS, U23.PD5(PCINT21/OC0B/T1)
- net CS_BIAS_DAC_3: now also U21.PB10/I2C2_SCL, U9A.CS; no longer U23.PD6(PCINT22/OC0A/AIN0), U24A.CS
- net CS_BIAS_DAC_4: now also U10A.CS, U21.PB11/I2C2_SDA/EVENTOUT; no longer U23.PD7(PCINT23/AIN1), U25A.CS
- net CS_DAC_1: now also U21.PA8/USART1_CK/TIM1_CH1/EVENTOUT/MCO, U5.!CS; no longer U23.PD0(RXD/PCINT16), U6.!CS
- net CS_DAC_2: now also U21.PA9/USART1_TX/TIM1_CH2/TIM15_BKIN, U6.!CS; no longer U23.PD1(TXD/PCINT17), U7.!CS
- net CS_DAC_3: now also U13.!CS, U21.PA10/USART1_RX/TIM1_CH3/TIM17_BKIN; no longer U15.!CS, U23.PD2(INT0/PCINT18)
- net CS_DAC_4: now also U14.!CS, U21.PA11/USART1_CTS/TIM1_CH4/EVENTOUT; no longer U16.!CS, U23.PD3(PCINT19/OC2B/INT1)
- net GND: now also C10.2, C11.2, C12.2, C14.2, C26.1, C27.1, C34.1, C36.GND, C37.-, C38.+, C39.-, C40.2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; no longer C10.1, C14.1, C21.2, C22.2, C26.2, C27.2, C32.2, C33.2, C34.2, C36.2, C37.1, C38.1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
- net MISO: now also U21.PB4/SPI1_MISO/TIM3_CH1/EVENTOUT; no longer ISP1.MISO, U23.(PCINT4/MISO)PB4
- net MOSI: now also U10A.SDI, U13.SDI, U14.SDI, U1A.SDI, U21.PB5/SPI1_MOSI/I2C1_SMBA/TIM16_BKIN/TIM3_CH2, U2A.SDI, U5.SDI, U9A.SDI; no longer ISP1.MOSI, U15.SDI, U16.SDI, U19A.SDI, U20A.SDI, U23.(PCINT3/OC2A/MOSI)PB3, U24A.SDI, U25A.SDI, U7.SDI
- net N$1: now also R13.1, U5.VOUT_A; no longer R30.1, U6.VOUT_A
- net N$10: now also R14.1, U5.VOUT_B; no longer R31.1, U6.VOUT_B
- net N$11: now also C20.1, R67.2, R68.2, R74.1, U18A.-IN; no longer C12.1, R2.2, R23.2, R24.2, R27.1, U5A.-IN
- net N$14: now also R16.2, R24.1, U7A.+IN; no longer R93.1, U19A.VOUTA
- net N$15: now also R77.1, R81.2, U17B.+IN; no longer R25.1, R28.2, U4B.+IN
- net N$16: now also R15.2, R21.2, U7B.+IN; no longer R94.1, U19A.VOUTB
- net N$17: now also R78.1, R82.2, U18B.+IN; no longer R37.1, R40.2, U5B.+IN
- net N$19: now also R12.1, R7.2, R8.2, U4B.-IN; no longer R15.2, R16.2, R20.1, U3B.-IN
- net N$2: now also R10.1, R3.2, R4.2, U3B.-IN; no longer R11.2, R12.2, R18.1, U2B.-IN
- net N$20: now also R12.2, U4B.OUT, U6.VREFB; no longer R20.2, U3B.OUT, U7.VREFB
- net N$21: now also R11.2, U4A.OUT, U6.VREFA; no longer R19.2, U3A.OUT, U7.VREFA
- net N$22: now also R11.1, R5.2, R6.2, U4A.-IN; no longer R13.2, R14.2, R19.1, U3A.-IN
- net N$23: now also R17.1, U6.VOUT_A; no longer R34.1, U7.VOUT_A
- net N$24: now also R17.2, R26.1, U8A.-IN; no longer R33.2, R34.2, R39.1, U9A.-IN
- net N$25: now also R26.2, R31.1, U8A.OUT; no longer R39.2, R48.1, U9A.OUT
- net N$26: now also R18.2, R28.1, U8B.-IN; no longer R35.2, R36.2, R42.1, U9B.-IN
- net N$27: now also R18.1, U6.VOUT_B; no longer R35.1, U7.VOUT_B
- net N$28: now also R28.2, R32.1, U8B.OUT; no longer R42.2, R52.1, U9B.OUT
- net N$29: now also R35.2, R36.2, R42.1; no longer R57.2, R58.2, R66.1
- net N$3: now also R13.2, R23.1, U7A.-IN; no longer R29.2, R30.2, R38.1, U8A.-IN
- net N$30: now also R42.2, U13.VREFB; no longer R66.2, U15.VREFB
- net N$31: now also R41.2, U13.VREFA; no longer R65.2, U15.VREFA
- net N$32: now also C19.1, R65.2, R66.2, R73.1, U17A.-IN; no longer C11.1, R114.2, R21.2, R22.2, R26.1, U4A.-IN
- net N$33: now also R33.2, R34.2, R41.1; no longer R55.2, R56.2, R65.1
- net N$34: now also R45.1, U13.VOUT_A; no longer R78.1, U15.VOUT_A
- net N$35: now also R45.2, R57.1, U15A.-IN; no longer R77.2, R78.2, R85.1, U17A.-IN
- net N$36: now also R57.2, R61.1, U15A.OUT; no longer R85.2, R89.1, U17A.OUT
- net N$37: now also R46.2, R59.1, U15B.-IN; no longer R79.2, R80.2, R87.1, U17B.-IN
- net N$38: now also R46.1, U13.VOUT_B; no longer R79.1, U15.VOUT_B
- net N$39: now also R59.2, R63.1, U15B.OUT; no longer R87.2, R91.1, U17B.OUT
- net N$4: now also R9.2, U3A.OUT, U5.VREFA; no longer R17.2, U2A.OUT, U6.VREFA
- net N$40: now also R39.2, R40.2, R44.1; no longer R61.2, R62.2, R68.1
- net N$41: now also R44.2, U14.VREFB; no longer R68.2, U16.VREFB
- net N$44: now also R43.2, U14.VREFA; no longer R67.2, U16.VREFA
- net N$46: now also R37.2, R38.2, R43.1; no longer R59.2, R60.2, R67.1
- net N$47: now also C36.+12V; no longer C55.+12V
- net N$48: now also C36.-12V; no longer C55.-12V
- net N$49: now also R48.1, U14.VOUT_A; no longer R82.1, U16.VOUT_A
- net N$5: now also R10.2, U3B.OUT, U5.VREFB; no longer R18.2, U2B.OUT, U6.VREFB
- net N$50: now also R48.2, R58.1, U16A.-IN; no longer R81.2, R82.2, R86.1, U18A.-IN
- net N$51: now also R58.2, R62.1, U16A.OUT; no longer R86.2, R90.1, U18A.OUT
- net N$52: now also R49.2, R60.1, U16B.-IN; no longer R83.2, R84.2, R88.1, U18B.-IN
- net N$53: now also R49.1, U14.VOUT_B; no longer R83.1, U16.VOUT_B
- net N$54: now also R60.2, R64.1, U16B.OUT; no longer R88.2, R92.1, U18B.OUT
- net N$55: now also C22.1, R76.1, U20A.-IN; no longer C20.1, R5.2, R74.1, U13A.-IN
- net N$59: now also C21.1, R75.1, U19A.-IN; no longer C19.1, R4.2, R73.1, U14A.-IN
- net N$6: now also R1.2, R2.2, R9.1, U3A.-IN; no longer R10.2, R17.1, R9.2, U2A.-IN
- net N$66: now also R79.1, R83.2, U19B.+IN; no longer R63.1, R64.2, U14B.+IN
- net N$67: now also R20.2, R27.1, U8A.+IN; no longer R95.1, U20A.VOUTA
- net N$68: now also R19.2, R22.1, U8B.+IN; no longer R96.1, U20A.VOUTB
- net N$69: now also R80.1, R84.2, U20B.+IN; no longer R75.1, R76.2, U13B.+IN
- net N$7: now also R25.2, R30.1, U7B.OUT; no longer R41.2, R51.1, U8B.OUT
- net N$70: now also R51.2, R53.2, U15A.+IN; no longer R101.1, U24A.VOUTA
- net N$71: now also R47.2, R54.2, U15B.+IN; no longer R102.1, U24A.VOUTB
- net N$72: now also R50.2, R56.2, U16B.+IN; no longer R103.1, U25A.VOUTA
- net N$73: now also R52.2, R55.2, U16A.+IN; no longer R104.1, U25A.VOUTB
- net N$75: now also C27.2, U21.PF1/OSC_OUT, X1.P$1; no longer R94.2, R98.1, U21B.-IN
- net N$76: now also C26.2, U21.PF0/OSC_IN, X1.P$2; no longer R95.2, R99.1, U22A.-IN
- net N$8: now also R23.2, R29.1, U7A.OUT; no longer R38.2, R47.1, U8A.OUT
- net N$9: now also R14.2, R25.1, U7B.-IN; no longer R31.2, R32.2, R41.1, U8B.-IN
- net OUT_L: now also C32.2, J19.2, JP2.1, R88.2, U22A.OUT; no longer C48.2, J17.2, R112.2, U28A.OUT
- net OUT_R: now also C33.2, JP2.2, R89.2, U22B.OUT; no longer C49.2, R113.2, U28B.OUT
- net PAN_CV_1: now also C19.2, R73.2, U17A.OUT, U21.PA4/SPI1_NSS/USART2_CK/TIM14_CH1/ADC_IN4; no longer C11.2, R26.2, U23.(ADC4/SDA/PCINT12)PC4, U4A.OUT
- net PAN_CV_2: now also C20.2, R74.2, U18A.OUT, U21.PA5/SPI1_SCK/ADC_IN5; no longer C12.2, R27.2, U23.(ADC5/SCL/PCINT13)PC5, U5A.OUT
- net PAN_CV_3: now also C21.2, R75.2, U19A.OUT, U21.PA6/SPI1_MISO/TIM3_CH1/TIM1_BKIN/TIM16_CH1/EVENTOUT/ADC_IN6; no longer C19.2, R73.2, U14A.OUT, U23.ADC6
- net PAN_CV_4: now also C22.2, R76.2, U20A.OUT, U21.PA7/SPI1_MOSI/TIM3_CH2/TIM14_CH1/TIM1_CH1N/TIM17_CH1/EVENTOUT/ADC_IN7; no longer C20.2, R74.2, U13A.OUT, U23.ADC7
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Other:
- note added: "Channel 1"
- note added: "Channel 1 PAN"
- note added: "Channel 1 VOL"
- note added: "Channel 2"
- note added: "Channel 2 PAN"
- note added: "Channel 2 VOL"
- note added: "Channel 3"
- note added: "Channel 3 PAN"
- note added: "Channel 3 VOL"
- note added: "Channel 4"
- note added: "Channel 4 PAN"
- note added: "Channel 4 VOL"
- note added: "Power"
- note removed: "PAN Input Normalizer:"
- note removed: "Volume CV Input Normalizer"

Commit message: Update jlcpcb-eagle
Parts:
- added SW1, SW2, SW3, SW4: (no value), jhbruhn-physical:SWITCH_PUSHBUTTON_LED
- D1, D2: value 1N4148W -> SS54; device jhbruhn-cdr:DIODE-SOD123 -> jhbruhn-cdr:DIODE-SMA
Changed lines of the file:
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@@
 <?xml version="1.0" encoding="utf-8"?>
 <!DOCTYPE eagle SYSTEM "eagle.dtd">
-<eagle version="9.5.2">
+<eagle version="9.6.0">
 <drawing>
 <settings>
@@
 <part name="R85" library="jhbruhn-cr" deviceset="R-EU_" device="R0402" package3d_urn="urn:adsk.eagle:package:23547/3" value="10k"/>
 <part name="+3V7" library="supply1" library_urn="urn:adsk.eagle:library:371" deviceset="+3V3" device=""/>
-<part name="D1" library="jhbruhn-cdr" deviceset="DIODE-" device="SOD123" package3d_urn="urn:adsk.eagle:package:43420/1" value="1N4148W"/>
-<part name="D2" library="jhbruhn-cdr" deviceset="DIODE-" device="SOD123" package3d_urn="urn:adsk.eagle:package:43420/1" value="1N4148W"/>
+<part name="D1" library="jhbruhn-cdr" deviceset="DIODE-" device="SMA" value="SS54"/>
+<part name="D2" library="jhbruhn-cdr" deviceset="DIODE-" device="SMA" value="SS54"/>
 <part name="X1" library="jhbruhn-cdr" deviceset="XTAL" device="NX5032" package3d_urn="urn:adsk.eagle:package:6240641/1" value="8MHz"/>
 <part name="JP2" library="jumper" library_urn="urn:adsk.eagle:library:252" deviceset="JP2E" device="" package3d_urn="urn:adsk.eagle:package:15452/1"/>
@@
 <part name="+3V17" library="supply1" library_urn="urn:adsk.eagle:library:371" deviceset="+3V3" device=""/>
 <part name="GND65" library="supply1" library_urn="urn:adsk.eagle:library:371" deviceset="GND" device=""/>
+<part name="SW1" library="jhbruhn-physical" deviceset="SWITCH_PUSHBUTTON_LED" device=""/>
+<part name="SW2" library="jhbruhn-physical" deviceset="SWITCH_PUSHBUTTON_LED" device=""/>
+<part name="SW3" library="jhbruhn-physical" deviceset="SWITCH_PUSHBUTTON_LED" device=""/>
+<part name="SW4" library="jhbruhn-physical" deviceset="SWITCH_PUSHBUTTON_LED" device=""/>
 </parts>
 <sheets>
@@
 <attribute name="VALUE" x="-33.02" y="-7.62" size="1.778" layer="96" rot="R90"/>
 </instance>
+<instance part="SW1" gate="SWITCH" x="27.94" y="35.56" smashed="yes">
+<attribute name="NAME" x="22.86" y="27.94" size="1.27" layer="95"/>
+</instance>
+<instance part="SW1" gate="LED" x="27.94" y="20.32" smashed="yes">
+<attribute name="NAME" x="31.496" y="15.748" size="1.778" layer="95" rot="R90"/>
+</instance>
+<instance part="SW2" gate="SWITCH" x="55.88" y="35.56" smashed="yes">
+<attribute name="NAME" x="50.8" y="27.94" size="1.27" layer="95"/>
+</instance>
+<instance part="SW2" gate="LED" x="55.88" y="20.32" smashed="yes">
+<attribute name="NAME" x="59.436" y="15.748" size="1.778" layer="95" rot="R90"/>
+</instance>
+<instance part="SW3" gate="SWITCH" x="83.82" y="35.56" smashed="yes">
+<attribute name="NAME" x="78.74" y="27.94" size="1.27" layer="95"/>
+</instance>
+<instance part="SW3" gate="LED" x="83.82" y="20.32" smashed="yes">
+<attribute name="NAME" x="87.376" y="15.748" size="1.778" layer="95" rot="R90"/>
+</instance>
+<instance part="SW4" gate="SWITCH" x="111.76" y="35.56" smashed="yes">
+<attribute name="NAME" x="106.68" y="27.94" size="1.27" layer="95"/>
+</instance>
+<instance part="SW4" gate="LED" x="111.76" y="20.32" smashed="yes">
+<attribute name="NAME" x="115.316" y="15.748" size="1.778" layer="95" rot="R90"/>
+</instance>
 </instances>
