File: stereo_mix/hardware_design/pcb/stereo_mix_back_digital.sch (EAGLE design)
At the start: 220 parts, among them IC1 4051CD4051, IC2 AMS1117-3.3, J1 WQP-PJ301M-12_JACK, J10 WQP-PJ301M-12_JACK, J11 WQP-PJ301M-12_JACK, J12 WQP-PJ301M-12_JACK, J13 WQP-PJ301M-12_JACK, J14 WQP-PJ301M-12_JACK, J15 WQP-PJ301M-12_JACK, J16 WQP-PJ301M-12_JACK, J17 CORTEX_DEBUG_PTH, J18 WQP-PJ301M-12_JACK, J19 WQP-PJ301M-12_JACK, J2 WQP-PJ301M-12_JACK, J3 WQP-PJ301M-12_JACK, J4 WQP-PJ301M-12_JACK, J5 WQP-PJ301M-12_JACK, J6 WQP-PJ301M-12_JACK, J7 WQP-PJ301M-12_JACK, J8 WQP-PJ301M-12_JACK, J9 WQP-PJ301M-12_JACK, U1 MCP4822E-SN, U10 MCP4822E-SN, U11 MCP6002T-I/SN, U12 MCP6002T-I/SN, U13 MCP4922E/SL, U14 MCP4922E/SL, U15 TL072CD, U16 TL072CD, U17 MCP6002T-I/SN, U18 MCP6002T-I/SN, U19 MCP6002T-I/SN, U2 MCP4822E-SN, U20 MCP6002T-I/SN, U21 STM32F030C8T6, U22 TL072CD, U3 MCP6002T-I/SN, U4 MCP6002T-I/SN, U5 MCP4922E/SL, U6 MCP4922E/SL, U7 TL072CD, U8 TL072CD, U9 MCP4822E-SN, X1 8MHz

Commit message: Fix problem in stereo_mix dac
Parts:
- C1, C10, C11, C12, C13, C14, C15, C16, C17, C18, C19, C2, C20, C21, C22, C23, C24, C25, C26, C27, C28, C29, C3, C30, C31, C32, C33, C34, C35, C4, C40, C42, C43, C44, C49, C5, C50, C53, C54, C55, C56, C57, C58, C59, C6, C60, C61, C62, C63, C64, C7, C8, C9: device jhbruhn-cr:C-EUC0402 -> jhbruhn-cdr:C-EUC0402

Commit message: Hardware filtering improvements
Parts:
- added C67, C68, C69, C70, C71, C72, C73, C74: 1uF, jhbruhn-cdr:C-EUC0402
- added R86, R87: 47k, jhbruhn-cdr:R-EU_R0402
- C49, C50, C53, C54, C55, C56: device jhbruhn-cdr:C-EUC0402 -> jhbruhn-cdr:C-EUC0805
- C51, C52: device jhbruhn-cr:C-EUC0402 -> jhbruhn-cdr:C-EUC0805
Connections:
- net BIAS_DAC1_L: now also C69.1
- net BIAS_DAC1_R: now also C70.1
- net BIAS_DAC2_L: now also C67.1
- net BIAS_DAC2_R: now also C68.1
- net BIAS_DAC3_L: now also C71.1
- net BIAS_DAC3_R: now also C72.1
- net BIAS_DAC4_L: now also C73.1
- net BIAS_DAC4_R: now also C74.1
- net GND: now also C67.2, C68.2, C69.2, C70.2, C71.2, C72.2, C73.2, C74.2, R86.1, R87.1
- net N$45: now also R86.2
- net N$57: now also R87.2

Commit message: Update stereo_mix to new hardware revision
Parts:
- removed C71, C72, C73, C74: 1uF, jhbruhn-cdr:C-EUC0402
- removed R84: 100k, jhbruhn-cr:R-EU_R0402
- removed SW1, SW2, SW3, SW4: (no value), jhbruhn-physical:SWITCH_PUSHBUTTON_LED
- added R100, R97, R98, R99: 20k, jhbruhn-cr:R-EU_R0402
- added R101: 120k, jhbruhn-cr:R-EU_R0402
- added S1, S2, S3, S4: (no value), jhbruhn-physical:TAC_SWITCHPTH
- added U$1, U$2, U$3, U$4: LED-BICOLOR-SHARED-THROUGHHOLE, jhbruhn-physical:LED-BICOLOR-SHARED-THROUGHHOLE
- C19, C20, C21, C22: value 4.7nF -> 1.0nF
- C67, C68, C69, C70: value 1uF -> 1.0nF
- R65, R67, R69, R71: value 200k -> 120k
- R73, R74, R75, R76: value 33k -> 20k
- R81, R82, R83: value 100k -> 120k
- VR1, VR2, VR3, VR4, VR5, VR6, VR7, VR8: value (none) -> 10k
Connections:
- removed net N$66: R79.1, R83.2, U19B.+IN
- removed net N$69: R80.1, R84.2, U20B.+IN
- new net LED_1_N: U$1.2, U21.PC14/OSC32_IN
- new net LED_2_N: U$2.2, U21.PC15/OSC32_OUT
- new net LED_3_N: U$3.2, U21.PF6/I2C2_SCL
- new net LED_4_N: U$4.2, U21.PF7/I2C2_SDA
- new net N$65: C67.1, R77.1, R81.2, R97.1, U17B.-IN
- new net N$74: C68.1, R78.1, R82.2, R98.1, U18B.-IN
- net AREF_-10: now also R101.1, R81.1, R82.1, R83.1
- net BIAS_DAC1_L: no longer C69.1
- net BIAS_DAC1_R: no longer C70.1
- net BIAS_DAC2_L: no longer C67.1
- net BIAS_DAC2_R: no longer C68.1
- net BIAS_DAC3_L: no longer C71.1
- net BIAS_DAC3_R: no longer C72.1
- net BIAS_DAC4_L: no longer C73.1
- net BIAS_DAC4_R: no longer C74.1
- net CS_DAC_1: now also U21.PA15/SPI1_NSS/USART2_RX/EVENTOUT; no longer U21.PA8/USART1_CK/TIM1_CH1/EVENTOUT/MCO
- net CS_DAC_2: now also U21.PB7/I2C1_SDA/USART1_RX/TIM17_CH1N; no longer U21.PA9/USART1_TX/TIM1_CH2/TIM15_BKIN
- net CS_DAC_3: now also U21.PB15/SPI2_MOSI/TIM1_CH3N/TIM15_CH1N/TIM15_CH2/RTC_REFIN; no longer U21.PA10/USART1_RX/TIM1_CH3/TIM17_BKIN
- net CS_DAC_4: now also U21.PC13/RTC_TAMP1/RTC_TS/RTC_OUT/WKUP2; no longer U21.PA11/USART1_CTS/TIM1_CH4/EVENTOUT
- net GND: now also S1.3, S1.4, S2.3, S2.4, S3.3, S3.4, S4.1, S4.2, U17B.+IN, U18B.+IN, U19B.+IN, U20B.+IN; no longer C67.2, C68.2, C69.2, C70.2, C71.2, C72.2, C73.2, C74.2, R81.1, R82.1, R83.1, R84.1, SW1LED.C, SW1SWITCH.2, SW1SWITCH.4, SW2LED.C, SW2SWITCH.2, SW2SWITCH.4, SW3LED.C, SW3SWITCH.2, SW3SWITCH.4, SW4LED.C, SW4SWITCH.2, SW4SWITCH.4
- net LED_1: now also U21.PA8/USART1_CK/TIM1_CH1/EVENTOUT/MCO; no longer U21.PB7/I2C1_SDA/USART1_RX/TIM17_CH1N
- net LED_2: now also U21.PA9/USART1_TX/TIM1_CH2/TIM15_BKIN; no longer U21.PB15/SPI2_MOSI/TIM1_CH3N/TIM15_CH1N/TIM15_CH2/RTC_REFIN
- net LED_3: now also U21.PA10/USART1_RX/TIM1_CH3/TIM17_BKIN; no longer U21.PC13/RTC_TAMP1/RTC_TS/RTC_OUT/WKUP2
- net LED_4: now also U21.PA11/USART1_CTS/TIM1_CH4/EVENTOUT; no longer U21.PC14/OSC32_IN
- net N$12: now also U$1.1; no longer SW1LED.A
- net N$13: now also U$2.1; no longer SW2LED.A
- net N$15: now also C69.1, R79.1, R83.2, R99.1, U19B.-IN; no longer R77.1, R81.2, U17B.+IN
- net N$17: now also C70.1, R100.1, R101.2, R80.1, U20B.-IN; no longer R78.1, R82.2, U18B.+IN
- net N$18: now also U$3.1; no longer SW3LED.A
- net N$42: now also U$4.1; no longer SW4LED.A
- net SWITCH_1: now also S1.1, S1.2; no longer SW1SWITCH.1, SW1SWITCH.3
- net SWITCH_2: now also S2.1, S2.2; no longer SW2SWITCH.1, SW2SWITCH.3
- net SWITCH_3: now also S3.1, S3.2; no longer SW3SWITCH.1, SW3SWITCH.3
- net SWITCH_4: now also S4.3, S4.4; no longer SW4SWITCH.1, SW4SWITCH.3
- net VOL_CV_1: now also C67.2, R97.2; no longer U17B.-IN
- net VOL_CV_2: now also C68.2, R98.2; no longer U18B.-IN
- net VOL_CV_3: now also C69.2, R99.2; no longer U19B.-IN
- net VOL_CV_4: now also C70.2, R100.2; no longer U20B.-IN
Other:
- note added: "+3V3 V Supply"
- note added: "-10V Reference"
- note added: "All Inputs -8.0V to 8.0V"
- note added: "Amplifier"
- note added: "MCU"
- note added: "Pots"
- note added: "Power Input"
- note added: "Power/Buffering"
- note added: "Programming"
- note added: "Switches/LEDs"
- moved on the sheet: C25, C26, C27, C28, C29, C30, C31, C34, C35, C40, D1, D2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
