File: midi2cv/hardware_design/pure_midi.sch (EAGLE design)
At the start: 92 parts, among them IC1 LD117AS50TR, IC2 74HCT125D, IC3 6N138SMD, IC4 74HCT125D, IC5 STM32F10XCXT6, IC6 LD117AS33TR, J1 CORTEX_DEBUG_PTH, SW1 EC12E_SW, U1 AD5676ARUZ, U2 AD5754BREZ, U3 TEXAS_INSTRUMENTS_LM4040C5IDB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, U4 MAX3421, U5 TEXAS_INSTRUMENTS_LM4040C25ID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, X1 OG-MIDI_MAB5SHCUI-SD-50BV, X2 KUSBVX, X3 OG-MIDI_MAB5SHCUI-SD-50BV, X4 KUSBVX-BS1N, X6 ABRACON_ABM3B-12.000MHZ-B2-TA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, X7 ABRACON_ABM3B-8.000MHZ-B2-TAB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

Commit message: Use newer processor for midi2cv, fix some hardware mistakes
Parts:
- removed DI1: OLED_1.3_128X64_SPI, microbuilder:OLED_1.3_128X64_SPI
- removed U$1, U$11, U$19, U$2, U$20, U$4, U$5, U$6, U$7, U$8: WQP-PJ301M-12_JACK, thonkiconn:WQP-PJ301M-12_JACK
- removed U5: TEXAS_INSTRUMENTS_LM4040C25IDBZRTEXAS_INSTRUMENTS_LM4040C25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, lm4040:TEXAS_INSTRUMENTS_LM4040C25IDBZRTEXAS_INSTRUMENTS_LM4040C25IDBZR_0_1
- added C18, C19, C20, C22: 22u, GMSN:CAPACITOR_POL-US153CLV-0505
- added C27, C28: 100n, rcl:C-EUC0603
- added D4: 1N4001, GMSN:DIODESMA
- added IC7: LD117AS50TR, v-reg:LD117AS50TR
- added R22: 33R, rcl:R-EU_R0603
- added R23, R30, R34, R38: 10k, rcl:R-EU_R0603
- added R24, R31, R35, R39: 56k, rcl:R-EU_R0603
- added R25, R28, R32, R36, R40: 39k, rcl:R-EU_R0603
- added R29, R33, R37: 1k, rcl:R-EU_R0603
- added X11, X12, X13, X14, X15, X16: WQP-PJ301M-12_JACK, thonkiconn:WQP-PJ301M-12_JACK
- added X21, X22: OG-MIDI_MAB5SHCUI-SD-50BV, yarns_v03:OG-MIDI_MAB5SHCUI-SD-50BV
- added X23: KUSBVX, con-kycon:KUSBVX
- added X24: ABRACON_ABM3B-12.000MHZ-B2-TABRACON_ABM3B-12.000MHZ-B2-T_0_0, Abracon - ABM3B-12.000MHZ-B2-T:ABRACON_ABM3B-12.000MHZ-B2-TABRACON_ABM3B-12.000MHZ-B2-T_0_0
- C1, C2, C7, C8: value 22p -> 100n
- C14, C15: value 100n -> 22p
- C21, C23: value 100n -> 22u; device rcl:C-EUC0603 -> GMSN:CAPACITOR_POL-US153CLV-0505
- C24, C25: value 100n -> 100nF
- C3, C4: value 22u -> 22p; device GMSN:CAPACITOR_POL-US153CLV-0505 -> rcl:C-EUC0603
- C5, C6: value 22u -> 100n; device GMSN:CAPACITOR_POL-US153CLV-0505 -> rcl:C-EUC0603
- D1: value 1N4148 -> OLED_1.3_128X64_SPI; device adafruit:DIODESOD-323F -> microbuilder:OLED_1.3_128X64_SPI
- D2: value 1N4001 -> 1N4148; device GMSN:DIODESMA -> adafruit:DIODESOD-323F
- IC1: value LD117AS50TR -> STM32F373C; device v-reg:LD117AS50TR -> og-stm32f2:STM32F373C
- IC2: value 74HCT125D -> AD5754BREZ; device 74xx-eu:74HCT125D -> ad5754:AD5754BREZ
- IC3: value 6N138SMD -> TL074D; device 6n138:6N138SMD -> linear:TL074D
- IC4: value 74HCT125D -> TL072D; device 74xx-eu:74HCT125D -> linear:TL072D
- IC5: value STM32F10XCXT6 -> 6N138SMD; device stm32:STM32F10XCXT6 -> 6n138:6N138SMD
- R1: value 1k -> 1k5
- R10: value 51R -> 1k
- R11: value 220R -> 1k
- R12: value 470R -> 10k
- R13: value 22R -> 56k
- R14: value 22R -> 39k
- R15: value 10k -> 1k; device resistor:R-EU_R0603 -> rcl:R-EU_R0603
- R16: value 10k -> 51R; device resistor:R-EU_R0603 -> rcl:R-EU_R0603
- R17: value 1k -> 220R
- R18: value 2k -> 51R
- R19: value 2k -> 1k
- R2, R3: value 4k7 -> 22R
- R20: value 1k5 -> 470R
- R21: value 10k -> 33R
- R26: value 33R -> 10k
- R27: value 33R -> 56k
- R4: value 1k -> 10k
- R5: value 1k -> 10k; device rcl:R-EU_R0603 -> resistor:R-EU_R0603
- R6, R7: value 1k -> 4k7
- R8: value 1k -> 2k
- R9: value 51R -> 2k
- U1: value AD5676ARUZ -> TEXAS_INSTRUMENTS_LM4040C5IDBZR1; device AD5676ARUZ:AD5676ARUZ -> lm4040:TEXAS_INSTRUMENTS_LM4040C5IDBZR1
- U2: value AD5754BREZ -> AD5676ARUZ; device ad5754:AD5754BREZ -> AD5676ARUZ:AD5676ARUZ
- U3: value TEXAS_INSTRUMENTS_LM4040C5IDBZR1 -> TEXAS_INSTRUMENTS_LM4040C25IDBZRTEXAS_INSTRUMENTS_LM4040C25IDBZR_0_1; device lm4040:TEXAS_INSTRUMENTS_LM4040C5IDBZR1 -> lm4040:TEXAS_INSTRUMENTS_LM4040C25IDBZRTEXAS_INSTRUMENTS_LM4040C25IDBZR_0_1
- X1: value OG-MIDI_MAB5SHCUI-SD-50BV -> ABRACON_ABM3B-8.000MHZ-B2-TABRACON_ABM3B-8.000MHZ-B2-T_0_0; device yarns_v03:OG-MIDI_MAB5SHCUI-SD-50BV -> Abracon - ABM3B-8.000MHZ-B2-T:ABRACON_ABM3B-8.000MHZ-B2-TABRACON_ABM3B-8.000MHZ-B2-T_0_0
- X2: value KUSBVX -> KUSBVX-BS1N; device con-kycon:KUSBVX -> con-kycon:KUSBVX-BS1N
- X3: value OG-MIDI_MAB5SHCUI-SD-50BV -> WQP-PJ301M-12_JACK; device yarns_v03:OG-MIDI_MAB5SHCUI-SD-50BV -> thonkiconn:WQP-PJ301M-12_JACK
- X4: value KUSBVX-BS1N -> WQP-PJ301M-12_JACK; device con-kycon:KUSBVX-BS1N -> thonkiconn:WQP-PJ301M-12_JACK
- X6: value ABRACON_ABM3B-12.000MHZ-B2-TABRACON_ABM3B-12.000MHZ-B2-T_0_0 -> WQP-PJ301M-12_JACK; device Abracon - ABM3B-12.000MHZ-B2-T:ABRACON_ABM3B-12.000MHZ-B2-TABRACON_ABM3B-12.000MHZ-B2-T_0_0 -> thonkiconn:WQP-PJ301M-12_JACK
- X7: value ABRACON_ABM3B-8.000MHZ-B2-TABRACON_ABM3B-8.000MHZ-B2-T_0_0 -> WQP-PJ301M-12_JACK; device Abracon - ABM3B-8.000MHZ-B2-T:ABRACON_ABM3B-8.000MHZ-B2-TABRACON_ABM3B-8.000MHZ-B2-T_0_0 -> thonkiconn:WQP-PJ301M-12_JACK
- renumbered U$12 to X8, U$13 to X9, U$14 to X10, U$15 to X17, U$16 to X18, U$17 to X19, U$18 to X20, U$3 to X5
Connections:
- removed net GATE_OUT_5: R7.1, U$19.2
- new net N$16: IC3A.-IN, R24.2, R25.1
- new net N$24: IC3C.+IN, R26.1
- new net N$25: IC3A.+IN, R23.1
- new net N$26: IC3D.OUT, R29.2, R31.1
- new net N$27: IC3D.-IN, R31.2, R32.1
- new net N$28: IC3D.+IN, R30.1
- new net N$29: IC4A.OUT, R33.2, R35.1
- new net N$30: IC4A.-IN, R35.2, R36.1
- new net N$31: IC4A.+IN, R34.1
- new net N$32: IC4B.OUT, R37.2, R39.1
- new net N$33: IC4B.-IN, R39.2, R40.1
- new net N$34: IC4B.+IN, R38.1
- new net N$35: R33.1, X15.2
- new net RST_DAC0: IC1.PB1/TIM3_CH4/ADC_IN9/SDADC1_AIN5P/SDADC1_AIN6M, U2.!RESET
- new net RST_OLED: D1.RES, IC1.PB0/SPI1_MOSI/I2S1_SD/TIM3_CH3/ADC_IN8/SDADC1_AIN6P
- net +12V: now also C10.1, C12.1, C18.+, C22.+, C23.+, C26.1, C9.1, D3.C, IC2.AVDD, IC3P.V+, IC4P.V+, IC7.IN, R8.2, R9.2, U2.VDD; no longer C11.1, C13.1, C3.+, D2.C, IC1.IN, R18.2, R19.2, U1.VDD, U2.AVDD
- net +3V3: now also C1.1, C17.1, C2.1, C20.+, C28.1, C5.1, C7.1, C8.1, D1.VCC, IC1.VBAT, IC1.VDDA, IC1.VDDSD, IC1.VDD_1, IC1.VDD_2, IC1.VREFSD+, IC2.DVCC, IC5.VCC, R1.1, R18.2, R20.2, R4.2, R5.2, R6.2, R7.2, U2.VLOGIC; no longer C14.1, C15.1, C21.1, C23.1, C24.1, C6.+, IC3.VCC, IC5AN_POWER.VBAT, IC5AN_POWER.VDDA, IC5POWER.VDD_1, IC5POWER.VDD_2, IC5POWER.VDD_3, R10.2, R12.2, R20.1, R21.2
- net +5V: now also C21.+, C24.1, IC7.OUT, X23.1; no longer C10.1, C12.1, C17.1, C5.+, C9.1, DI1.VCC, IC1.OUT, IC2P.VCC, IC4P.VCC, R15.2, R16.2, R2.2, R3.2, U1.VLOGIC, U2.DVCC, X2.1
- net -12V: now also C11.2, C13.2, C19.-, C27.2, D4.A, IC2.AVSS, IC2.AVSS_2, IC3P.V-, IC4P.V-; no longer C26.2, C4.-, D3.A, U2.AVSS, U2.AVSS_2
- net AREF_25: now also IC2.REFIN, R9.1, U3.CATHODE; no longer R18.1, U2.REFIN, U5.CATHODE
- net AREF_5: now also R8.1, U1.CATHODE, U2.VREF; no longer R19.1, U1.VREF, U3.CATHODE
- net CV_OUT_1: now also IC2.VOUTA, X3.2; no longer U$1.2, U2.VOUTA
- net CV_OUT_10: now also U2.VOUT5; no longer U1.VOUT5
- net CV_OUT_11: now also U2.VOUT6; no longer U1.VOUT6
- net CV_OUT_12: now also U2.VOUT7; no longer U1.VOUT7
- net CV_OUT_2: now also IC2.VOUTB, X4.2; no longer U$2.2, U2.VOUTB
- net CV_OUT_3: now also IC2.VOUTC; no longer U2.VOUTC
- net CV_OUT_4: now also IC2.VOUTD, X6.2; no longer U$4.2, U2.VOUTD
- net CV_OUT_5: now also U2.VOUT0, X7.2; no longer U$11.2, U1.VOUT0
- net CV_OUT_6: now also U2.VOUT1; no longer U1.VOUT1
- net CV_OUT_7: now also U2.VOUT2; no longer U1.VOUT2
- net CV_OUT_8: now also U2.VOUT3; no longer U1.VOUT3
- net CV_OUT_9: now also U2.VOUT4; no longer U1.VOUT4
- net D_GATE_OUT_1: now also IC1.PA0/USART2_CTS/TIM2_CH1/TIM5_CH1/ADC_IN0, R23.2; no longer IC2A.I, IC5PORTA_L.PA0
- net D_GATE_OUT_2: now also IC1.PA1/SPI3_SCK/I2S3_CK/USART2_RTS/TIM2_CH2/TIM5_CH2/ADC_IN1, R12.2; no longer IC2B.I, IC5PORTA_L.PA1
- net D_GATE_OUT_3: now also IC1.PA2/SPI3_MISO/I2S3_MCK/USART2_TX/TIM2_CH3/TIM5_CH3/ADC_IN2, R26.2; no longer IC2C.I, IC5PORTA_L.PA2
- net D_GATE_OUT_4: now also IC1.PA3/SPI3_MOSI/I2S3_SD/USART2_RX/TIM2_CH4/TIM5_CH4/ADC_IN3, R30.2; no longer IC2D.I, IC5PORTA_L.PA3
- net D_GATE_OUT_5: now also IC1.PA4/SPI1_NSS/I2S1_WS/SPI3_NSS/I2S3_WS/USART2_CK/TIM3_CH2/ADC_IN4/DAC1_OUT1, R34.2; no longer IC4C.I, IC5PORTA_L.PA4
- net D_GATE_OUT_6: now also IC1.PA5/SPI1_SCK/I2S1_CK/TIM2_CH1/ADC_IN5/DAC1_OUT2, R38.2; no longer IC4D.I, IC5PORTA_L.PA5
- net ENC_A: now also IC1.PC13/TIMESTAMP/RTC_TAMPER1; no longer IC5PORTC.PC13, R15.1
- net ENC_B: now also IC1.PC14/OSC32_IN; no longer IC5PORTC.PC14, R16.1
- net ENC_SW: now also IC1.PC15/OSC32_OUT; no longer IC5PORTC.PC15
- net GATE_OUT_1: now also R10.1, X11.2; no longer R1.1, U$5.2
- net GATE_OUT_2: now also R11.1, X12.2; no longer R4.1, U$6.2
- net GATE_OUT_3: now also R15.1, X13.2; no longer R5.1, U$7.2
- net GATE_OUT_4: now also R29.1, X14.2; no longer R6.1, U$8.2
- net GATE_OUT_6: now also R37.1, X16.2; no longer R8.1, U$20.2
- net GND: now also C1.2, C11.1, C13.1, C14.1, C15.1, C18.-, C19.+, C2.2, C20.-, C21.-, C22.-, C23.-, C26.2, C27.1, C28.2, C3.1, C4.1, C5.2, C6.2, C7.2, C8.2, D1.GND, IC1.BOOT0, IC1.VSSA, IC1.VSSSD/VREFSD-, IC1.VSS_1, IC2.BIN/_2SCOMP, IC2.DAC_GND, IC2.DAC_GND_2, IC2.GND, IC2.LDAC, IC2.SIG_GND, IC2.SIG_GND_2, IC5.GND, IC7.ADJ, R14.2, R19.1, R25.2, R28.2, R32.2, R36.2, R40.2, U1.ANODE, U2.!LDAC, U2.RSTSEL, X1.1_GND, X1.2_GND, X11.1, X12.1, X13.1, X14.1, X15.1, X16.1, X22.2, X23.4, X23.S1, X23.S2, X24.1_GND, X24.2_GND, X3.1, X4.1, X6.1, X7.1; no longer C1.1, C11.2, C13.2, C14.2, C15.2, C2.1, C21.2, C23.2, C26.1, C3.-, C4.+, C5.-, C6.-, C7.1, C8.1, DI1.GND, IC1.ADJ, IC2A.OE, IC2B.OE, IC2C.OE, IC2D.OE, IC2P.GND, IC3.GND, IC4C.OE, IC4D.OE, IC4P.GND, IC5AN_POWER.VSSA, IC5PORTB_L.PB2, IC5POWER.VSS_1, IC5POWER.VSS_2, IC5POWER.VSS_3, IC5RESET.BOOT0, R17.1, U$1.1, U$11.1, U$19.1, U$2.1, U$20.1, U$4.1, U$5.1, U$6.1, U$7.1, U$8.1, U1.!LDAC, U1.GND, U1.RSTSEL, U2.BIN/_2SCOMP, U2.DAC_GND, U2.DAC_GND_2, U2.LDAC, U2.SIG_GND, U2.SIG_GND_2, U5.ANODE, X3.2, X4.4, X4.S1, X4.S2, X6.1_GND, X6.2_GND, X7.1_GND, X7.2_GND
- net INT_USB: now also IC1.PE8/SDADC1_AIN8P/SDADC2_AIN8P; no longer IC5PORTB_H.PB10
- net JTCK: now also IC1.PA14/I2C1_SDA/JTCK-SWCLK; no longer IC5PORTA_H.PA14
- net JTDI: now also IC1.PA15/SPI1_NSS/I2S1_WS/SPI3_NSS/I2S3_WS/I2C1_SCL/TIM2_CH1_ETR/JTDI; no longer IC5PORTA_H.PA15
- net JTDO: now also IC1.PB3/SPI1_SCK/I2S1_CK/SPI3_SCK/I2S3_CK/USART2_TX/TIM2_CH2/JTDO/SPI3_SCK/JTDO; no longer IC5PORTB_L.PB3
- net JTMS: now also IC1.PA13/SPI1_MISO/I2S1_MCK/USART3_CTS/TIM4_CH3/TIM5_CH4/JTMS-SWDIO; no longer IC5PORTA_H.PA13
- net MIDI_DATA_IN: now also IC1.PA10/SPI2_MOSI/I2S2_SD/I2C2_SDA/USART1_RX/TIM2_CH4, IC5.VO, R20.1; no longer IC3.VO, IC5PORTA_H.PA10, R12.1
- net MIDI_DATA_OUT: now also IC1.PA9/SPI_MISO/I2S2_MCK/I2C2_SCL/USART1_TX/TIM2_CH3, R16.1; no longer IC5PORTA_H.PA9, R9.1
- net MISO: now also IC1.PB14/SPI2_MISO/I2S2_MCK/USART3_RTS/SDADC3_AIN8P; no longer IC5PORTB_H.PB14
- net MOSI: now also D1.MOSI, IC1.PB15/SPI2_MOSI/I2S2_SD/SDADC3_AIN7P/SDADC3_AIN8M, IC2.SDIN, U2.SDI; no longer DI1.MOSI, IC5PORTB_H.PB15, U1.SDI, U2.SDIN
- net N$1: now also R7.1, U2.GAIN; no longer R2.1, U1.GAIN
- net N$10: now also IC3A.OUT, R10.2, R24.1; no longer IC2A.O, R1.2
- net N$11: now also IC3B.OUT, R11.2, R13.1; no longer IC2B.O, R4.2
- net N$12: now also IC5.VB, R19.2; no longer IC3.VB, R17.2
- net N$13: now also D3.A; no longer D2.A
- net N$14: now also IC3B.-IN, R13.2, R14.1; no longer IC2C.O, R5.2
- net N$15: now also IC3B.+IN, R12.1; no longer IC2D.O, R6.2
- net N$17: now also IC3C.OUT, R15.2, R27.1; no longer IC4C.O, R7.2
- net N$18: now also IC3C.-IN, R27.2, R28.1; no longer IC4D.O, R8.2
- net N$19: now also R16.2, X22.5; no longer R9.2, X3.5
- net N$2: now also IC2.CLR, R6.1; no longer R3.1, U2.CLR
- net N$20: now also D4.C; no longer D3.C
- net N$21: now also R2.1, X2.2; no longer R13.1, X4.2
- net N$22: now also R18.1, X22.4; no longer R10.1, X3.4
- net N$23: now also R1.2, R3.1, X2.3; no longer R14.1, R20.2, X4.3
- net N$3: now also C4.2, IC1.PF1/OSC_OUT/I2C2_SCL, X1.X2; no longer C2.2, IC5PORTD/OSC.PD1/OSC=>, X7.X2
- net N$4: now also D2.C, IC5.A, R17.2; no longer D1.C, IC3.A, R11.2
- net N$5: now also R17.1, X21.4; no longer R11.1, X1.4
- net N$6: now also C3.2, IC1.PF0/OSC_IN/I2C2_SDA, X1.X1; no longer C1.2, IC5PORTD/OSC.PD0/OSC<=, X7.X1
- net N$7: now also C14.2, X24.X1; no longer C8.2, X6.X1
- net N$8: now also C15.2, X24.X2; no longer C7.2, X6.X2
- net N$9: now also D2.A, IC5.C, X21.5; no longer D1.A, IC3.C, X1.5
- net RST: now also C6.1, IC1.NRST, R4.1; no longer DI1.RES, IC5RESET.NRST, R21.1, U1.!RESET
- net RST_USB: now also IC1.PB6/I2C1_SCL/USART1_TX/TIM4_CH1; no longer IC5PORTB_H.PB8
- net SCK: now also D1.CLK, IC1.PB8/SPI2_SCK/I2S2_CK/I2C1_SCL/USART3_TX/CAN_RX/TIM4_CH3, IC2.SCLK; no longer DI1.CLK, IC5PORTB_H.PB13, U1.SCLK
- net SDC_OLED: now also D1.SDC, IC1.PB9/SPI2_NSS/I2S2_WS/I2C1_SDA/USART3_RX/CAN_TX/TIM4_CH4; no longer DI1.SDC, IC5PORTB_H.PB12
- net SS_DAC0: now also IC1.PB4/SPI1_MISO/I2S1_MCK/SPI3_MISO/I2S3_MCK/USART2_RX/TIM3_CH1/NJTRST, U2.!SYNC; no longer IC5PORTB_L.PB6, U1.!SYNC
- net SS_DAC1: now also IC1.PB5/SPI1_MOSI/I2S1_SD/SPI3_MOSI/I2S3_SD/I2C1_SMBAI/USART2_CK/TIM3_CH2, IC2.SYNC; no longer IC5PORTB_L.PB7, U2.SYNC
- net SS_OLED: now also D1.CCS, IC1.PB2/SDADC1_AIN4P/SDADC2_AIN6P, R5.1; no longer DI1.CCS, IC5PORTB_H.PB11
- net SS_USB: now also IC1.PB7/I2C1_SDA/USART1_RX/TIM4_CH2; no longer IC5PORTB_H.PB9
- net USB_D_N: now also R22.1, X23.2; no longer R26.1, X2.2
- net USB_D_P: now also R21.1, X23.3; no longer R27.1, X2.3
- net USB_N: now also R22.2; no longer R26.2
- net USB_P: now also R21.2; no longer R27.2
- net USB_PER_D_N: now also IC1.PA11/SPI2_NSS/I2S2_WS/SPI1_NSS/I2S1_WS/USART1_CTS/CAN_RX/TIM4_CH1/TIM5_CH2, R2.2; no longer IC5PORTA_H.PA11, R13.2
- net USB_PER_D_P: now also IC1.PA12/SPI1_SCK/I2S1_CK/USART1_RTS/CAN_TX/TIM4_CH2/TIM5_CH3, R3.2; no longer IC5PORTA_H.PA12, R14.2

Commit message: Use some sweet ass voltage references
Parts:
- removed R8, R9: 2k, rcl:R-EU_R0603
- removed U1: TEXAS_INSTRUMENTS_LM4040C5IDBZR1, lm4040:TEXAS_INSTRUMENTS_LM4040C5IDBZR1
- removed U3: TEXAS_INSTRUMENTS_LM4040C25IDBZRTEXAS_INSTRUMENTS_LM4040C25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, lm4040:TEXAS_INSTRUMENTS_LM4040C25IDBZRTEXAS_INSTRUMENTS_LM4040C25IDBZR_0_1
- added C29, C30, C31, C32: 100n, rcl:C-EUC0603
- added IC8: ADR435, analog-adr43x:ADR43XXRMZ
- added IC9: ADR431, analog-adr43x:ADR43XXRMZ
Connections:
- net +12V: now also C29.1, C30.1, IC8.VIN, IC9.VIN; no longer R8.2, R9.2
- net AREF_25: now also C32.1, IC9.VOUT; no longer R9.1, U3.CATHODE
- net AREF_5: now also C31.1, IC8.VOUT; no longer R8.1, U1.CATHODE
- net GND: now also C29.2, C30.2, C31.2, C32.2, IC8.GND, IC9.GND; no longer U1.ANODE, U3.ANODE

Commit message: Last layout improvements
Parts:
- R21, R22: value 33R -> 22R
- R6, R7: value 4k7 -> 10k
Changed lines of the file:
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@@
 <part name="GND23" library="supply1" library_urn="urn:adsk.eagle:library:371" deviceset="GND" device=""/>
 <part name="P+3" library="supply1" library_urn="urn:adsk.eagle:library:371" deviceset="+12V" device=""/>
-<part name="R7" library="rcl" library_urn="urn:adsk.eagle:library:334" deviceset="R-EU_" device="R0603" package3d_urn="urn:adsk.eagle:package:23555/3" value="4k7"/>
+<part name="R7" library="rcl" library_urn="urn:adsk.eagle:library:334" deviceset="R-EU_" device="R0603" package3d_urn="urn:adsk.eagle:package:23555/3" value="10k"/>
 <part name="X3" library="thonkiconn" deviceset="WQP-PJ301M-12_JACK" device=""/>
 <part name="X4" library="thonkiconn" deviceset="WQP-PJ301M-12_JACK" device=""/>
@@
 <part name="X23" library="con-kycon" library_urn="urn:adsk.eagle:library:157" deviceset="KUSBVX" device="" package3d_urn="urn:adsk.eagle:package:7682/1"/>
 <part name="GND48" library="supply1" library_urn="urn:adsk.eagle:library:371" deviceset="GND" device=""/>
-<part name="R22" library="rcl" library_urn="urn:adsk.eagle:library:334" deviceset="R-EU_" device="R0603" package3d_urn="urn:adsk.eagle:package:23555/3" value="33R"/>
-<part name="R21" library="rcl" library_urn="urn:adsk.eagle:library:334" deviceset="R-EU_" device="R0603" package3d_urn="urn:adsk.eagle:package:23555/3" value="33R"/>
+<part name="R22" library="rcl" library_urn="urn:adsk.eagle:library:334" deviceset="R-EU_" device="R0603" package3d_urn="urn:adsk.eagle:package:23555/3" value="22R"/>
+<part name="R21" library="rcl" library_urn="urn:adsk.eagle:library:334" deviceset="R-EU_" device="R0603" package3d_urn="urn:adsk.eagle:package:23555/3" value="22R"/>
 <part name="GND49" library="supply1" library_urn="urn:adsk.eagle:library:371" deviceset="GND" device=""/>
 <part name="GND52" library="supply1" library_urn="urn:adsk.eagle:library:371" deviceset="GND" device=""/>
@@
 <part name="P-1" library="supply1" library_urn="urn:adsk.eagle:library:371" deviceset="-12V" device=""/>
 <part name="P+1" library="supply1" library_urn="urn:adsk.eagle:library:371" deviceset="+12V" device=""/>
-<part name="R6" library="rcl" library_urn="urn:adsk.eagle:library:334" deviceset="R-EU_" device="R0603" package3d_urn="urn:adsk.eagle:package:23555/3" value="4k7"/>
+<part name="R6" library="rcl" library_urn="urn:adsk.eagle:library:334" deviceset="R-EU_" device="R0603" package3d_urn="urn:adsk.eagle:package:23555/3" value="10k"/>
 <part name="GND16" library="supply1" library_urn="urn:adsk.eagle:library:371" deviceset="GND" device=""/>
 <part name="GND15" library="supply1" library_urn="urn:adsk.eagle:library:371" deviceset="GND" device=""/>

Commit message: Remove usb from midi
Parts:
- removed C16, C17: 100n, rcl:C-EUC0603
- removed C21, C23: 22u, GMSN:CAPACITOR_POL-US153CLV-0505
- removed C24: 100nF, rcl:C-EUC0603
- removed FD1, FD2, FD3, FD4: FIDUCIALUFIDUCIAL, SparkFun-Aesthetics:FIDUCIALUFIDUCIAL
- removed IC3: TL074D, linear:TL074D
- removed R21, R22: 22R, rcl:R-EU_R0603
- removed U4: MAX3421, SparkFun-IC-Comms:MAX3421ESMD
- removed X23: KUSBVX, con-kycon:KUSBVX
- removed X24: ABRACON_ABM3B-12.000MHZ-B2-TABRACON_ABM3B-12.000MHZ-B2-T_0_0, Abracon - ABM3B-12.000MHZ-B2-T:ABRACON_ABM3B-12.000MHZ-B2-TABRACON_ABM3B-12.000MHZ-B2-T_0_0
- added IC10: TL072CD, jhbruhn-opamp:TL072CD
- C1, C10, C11, C12, C13, C2, C25, C26, C27, C28, C29, C3, C30, C31, C32, C4, C5, C6, C7, C8, C9: device rcl:C-EUC0603 -> jhbruhn-cdr:C-EUC0603
- C14, C15: value 22p -> 100n; device rcl:C-EUC0603 -> jhbruhn-cdr:C-EUC0603
- C18, C19, C20, C22: value 22u -> 10uF; device GMSN:CAPACITOR_POL-US153CLV-0505 -> jhbruhn-cdr:CPOL-EUA/3216-18R
- D2: value 1N4148 -> 1N4148W; device adafruit:DIODESOD-323F -> jhbruhn-cdr:DIODE-SOD123
- D3, D4: value 1N4001 -> B5819W; device GMSN:DIODESMA -> jhbruhn-cdr:DIODE-SOD123
- IC4: value TL072D -> TL072CD; device linear:TL072D -> jhbruhn-opamp:TL072CD
- IC7: value LD117AS50TR -> TL072CD; device v-reg:LD117AS50TR -> jhbruhn-opamp:TL072CD
- R1, R10, R11, R12, R13, R14, R15, R16, R17, R18, R19, R2, R20, R23, R24, R25, R26, R27, R28, R29, R3, R30, R31, R32, R33, R34, R35, R36, R37, R38, R39, R4, R40, R6, R7: device rcl:R-EU_R0603 -> jhbruhn-cdr:R-EU_R0603
- R5: device resistor:R-EU_R0603 -> jhbruhn-cdr:R-EU_R0603
- X1: value ABRACON_ABM3B-8.000MHZ-B2-TABRACON_ABM3B-8.000MHZ-B2-T_0_0 -> 8MHz; device Abracon - ABM3B-8.000MHZ-B2-T:ABRACON_ABM3B-8.000MHZ-B2-TABRACON_ABM3B-8.000MHZ-B2-T_0_0 -> jhbruhn-cdr:XTALNX5032
Connections:
- removed net +5V: C21.+, C24.1, IC7.OUT, X23.1
- removed net N$7: C14.2, U4.X0, X24.X1
- removed net USB_D_N: R22.1, X23.2
- removed net USB_D_P: R21.1, X23.3
- removed net USB_N: R22.2, U4.D-
- removed net USB_P: R21.2, U4.D+
- net +12V: now also C14.1, IC10P.V+, IC7P.V+; no longer C23.+, IC3P.V+, IC7.IN
- net +3V3: no longer C16.1, C17.1, U4.VCC, U4.VL
- net -12V: now also C15.2, IC10P.V-, IC7P.V-; no longer IC3P.V-
- net GND: now also C14.2; no longer C14.1, C16.2, C17.2, C18.-, C19.+, C21.-, C23.-, C24.2, IC7.ADJ, PWR1.3, PWR1.4, PWR1.5, PWR1.6, PWR1.7, PWR1.8, U4.GND@19, U4.GND@3, X1.1_GND, X1.2_GND, X23.4, X23.S1, X23.S2, X24.1_GND, X24.2_GND
- net INT_USB: no longer U4.INT
- net MISO: no longer U4.MISO
- net MOSI: no longer U4.MOSI
- net N$10: now also IC10A.OUT; no longer IC3A.OUT
- net N$11: now also IC10B.OUT; no longer IC3B.OUT
- net N$14: now also IC10B.-IN; no longer IC3B.-IN
- net N$15: now also IC10B.+IN; no longer IC3B.+IN
- net N$16: now also IC10A.-IN; no longer IC3A.-IN
- net N$17: now also IC7A.OUT; no longer IC3C.OUT
- net N$18: now also IC7A.-IN; no longer IC3C.-IN
- net N$24: now also IC7A.+IN; no longer IC3C.+IN
- net N$25: now also IC10A.+IN; no longer IC3A.+IN
- net N$26: now also IC7B.OUT; no longer IC3D.OUT
- net N$27: now also IC7B.-IN; no longer IC3D.-IN
- net N$28: now also IC7B.+IN; no longer IC3D.+IN
- net N$3: now also X1.P$1; no longer X1.X2
- net N$6: now also X1.P$2; no longer X1.X1
- net N$8: now also C18.-, C19.+, PWR1.3, PWR1.4, PWR1.5, PWR1.6, PWR1.7, PWR1.8; no longer C15.2, U4.X1, X24.X2
- net RST_USB: no longer U4.RES
- net SCK: no longer U4.SCK
- net SS_USB: no longer U4.SS
