File: deprecated/midi2cv/hardware_design/pure_midi.sch (EAGLE design)
At the start: 103 parts, among them IC1 STM32F373C, IC10 TL072CD, IC2 AD5754BREZ, IC4 TL072CD, IC5 6N138SMD, IC6 LD117AS33TR, IC7 TL072CD, IC8 ADR435, IC9 ADR431, J1 CORTEX_DEBUG_PTH, SW1 EC12E_SW, U2 AD5676ARUZ, X1 8MHz, X10 WQP-PJ301M-12_JACK, X11 WQP-PJ301M-12_JACK, X12 WQP-PJ301M-12_JACK, X13 WQP-PJ301M-12_JACK, X14 WQP-PJ301M-12_JACK, X15 WQP-PJ301M-12_JACK, X16 WQP-PJ301M-12_JACK, X17 WQP-PJ301M-12_JACK, X18 WQP-PJ301M-12_JACK, X19 WQP-PJ301M-12_JACK, X2 KUSBVX-BS1N, X20 WQP-PJ301M-12_JACK, X21 OG-MIDI_MAB5SHCUI-SD-50BV, X22 OG-MIDI_MAB5SHCUI-SD-50BV, X3 WQP-PJ301M-12_JACK, X4 WQP-PJ301M-12_JACK, X5 WQP-PJ301M-12_JACK, X6 WQP-PJ301M-12_JACK, X7 WQP-PJ301M-12_JACK, X8 WQP-PJ301M-12_JACK, X9 WQP-PJ301M-12_JACK

Commit message: Move midi2cv to deprecated folder
Parts:
- added U$1: LED-BICOLOR-SHARED-THROUGHHOLE, jhbruhn-physical:LED-BICOLOR-SHARED-THROUGHHOLE
Connections:
- removed net RST_USB: IC1.PB6/I2C1_SCL/USART1_TX/TIM4_CH1
- removed net SS_USB: IC1.PB7/I2C1_SDA/USART1_RX/TIM4_CH2
Changed lines of the file:
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@@
 <part name="C15" library="jhbruhn-cdr" deviceset="C-EU" device="C0603" package3d_urn="urn:adsk.eagle:package:23616/2" value="100n"/>
 <part name="X1" library="jhbruhn-cdr" deviceset="XTAL" device="NX5032" package3d_urn="urn:adsk.eagle:package:6240641/1" value="8MHz"/>
+<part name="U$1" library="jhbruhn-physical" deviceset="LED-BICOLOR-SHARED-THROUGHHOLE" device=""/>
 </parts>
 <sheets>
@@
 <pinref part="IC1" gate="G$$1" pin="PA3/SPI3_MOSI/I2S3_SD/USART2_RX/TIM2_CH4/TIM5_CH4/ADC_IN3"/>
 <label x="215.9" y="127" size="1.778" layer="95"/>
-</segment>
-</net>
-<net name="SS_USB" class="0">
-<segment>
-<wire x1="213.36" y1="68.58" x2="228.6" y2="68.58" width="0.1524" layer="91"/>
-<pinref part="IC1" gate="G$$1" pin="PB7/I2C1_SDA/USART1_RX/TIM4_CH2"/>
-<label x="215.9" y="68.58" size="1.778" layer="95"/>
-</segment>
-</net>
-<net name="RST_USB" class="0">
-<segment>
-<wire x1="213.36" y1="71.12" x2="228.6" y2="71.12" width="0.1524" layer="91"/>
-<pinref part="IC1" gate="G$$1" pin="PB6/I2C1_SCL/USART1_TX/TIM4_CH1"/>
-<label x="215.9" y="71.12" size="1.778" layer="95"/>
 </segment>
 </net>
@@
 <attribute name="VALUE" x="197.104" y="-55.499" size="1.778" layer="96"/>
 </instance>
+<instance part="U$1" gate="G$1" x="289.56" y="-38.1" smashed="yes">
+<attribute name="NAME" x="283.21" y="-32.258" size="1.778" layer="95"/>
+<attribute name="VALUE" x="283.21" y="-45.72" size="1.778" layer="95"/>
+</instance>
 </instances>
